File: microprocessor.kicad_sch (KiCad schematic)
At the start: 36 parts, among them J4 Conn_02x03_Odd_Even, U3 ATxmega192A3U-A, X1 ABLS-16.000MHZ-B4-T

Commit message: removed autosave file and corrected schematic electrical rules check warnings and errors
Connections:
- net 3.3V is gone; now on net +3.3V: R38.1
Changed lines of the file:
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@@
     )
   )
-  (global_label "3.3V" (shape input) (at 43.942 95.25 180) (fields_autoplaced)
+  (global_label "+3.3V" (shape input) (at 43.942 95.25 180) (fields_autoplaced)
     (effects (font (size 1.27 1.27)) (justify right))
-    (property "Intersheet References" "${INTERSHEET_REFS}" (id 0) (at 37.4165 95.1706 0)
+    (property "Intersheet References" "${INTERSHEET_REFS}" (id 0) (at 35.8441 95.1706 0)
       (effects (font (size 1.27 1.27)) (justify right) hide)
     )

Commit message: replaced some parts numbers with parts that are available
Parts:
- C69, C70: Model CL21C131JBANNNC -> 08055A131JAT2A
- U3: Model (none) -> ATxmega192A3U-A
Changed lines of the file:
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@@
+      (effects (font (size 1.27 1.27)) hide)
+    )
+    (property "Model" "ATxmega192A3U-A" (id 4) (at 116.332 103.378 0)
       (effects (font (size 1.27 1.27)) hide)
     )
@@
       (effects (font (size 1.27 1.27)) hide)
     )
-    (property "Model" "CL21C131JBANNNC" (id 4) (at 164.592 133.858 0)
+    (property "Model" "08055A131JAT2A" (id 4) (at 164.592 133.858 0)
       (effects (font (size 1.27 1.27)) hide)
     )
@@
       (effects (font (size 1.27 1.27)) hide)
     )
-    (property "Model" "CL21C131JBANNNC" (id 4) (at 184.404 117.602 0)
+    (property "Model" "08055A131JAT2A" (id 4) (at 184.404 117.602 0)
       (effects (font (size 1.27 1.27)) hide)
     )

Commit message: modified file to allow floating 5V buffer oe inputs until boot completes.
Parts:
- added R88, R89: 0, Resistor_SMD:R_0805_2012Metric_Pad1.20x1.40mm_HandSolder, symbol Device:R_US
- added TP23: test, Connector_PinHeader_1.00mm:PinHeader_1x01_P1.00mm_Vertical, symbol Connector:TestPoint
Connections:
- net GND: now also R88.1
- net at U3.51 (PF5): now also R89.2
- new net buffer_enable: R88.2, R89.1, TP23.1
- no-connect marks 3 -> 2
Other:
- note added: "Note 1 - populate either R88 or R89. If U5 pin 51 is programmed to go low after boot, populate R89. Otherwise populate R88."
Changed lines of the file:
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@@
     (comment 2 "Licensed under CERN-OHL-S v2 ")
   )
+  (junction (at 67.818 100.838) (diameter 0) (color 0 0 0 0)
+  )
   (junction (at 76.962 17.526) (diameter 0) (color 0 0 0 0)
   )
@@
   )
   (junction (at 188.214 123.698) (diameter 0) (color 0 0 0 0)
+  )
+  (junction (at 73.66 100.838) (diameter 0) (color 0 0 0 0)
   )
   (junction (at 216.154 43.688) (diameter 0) (color 0 0 0 0)
@@
   (no_connect (at 31.75 67.818))
   (no_connect (at 19.05 67.818))
-  (no_connect (at 98.552 100.838))
   (wire (pts (xy 67.31 121.158) (xy 67.31 122.428))
     (stroke (width 0) (type default) (color 0 0 0 0))
@@
     (stroke (width 0) (type default) (color 0 0 0 0))
   )
-  (wire (pts (xy 98.552 110.998) (xy 67.31 110.998))
-    (stroke (width 0) (type default) (color 0 0 0 0))
-  )
   (wire (pts (xy 134.112 77.978) (xy 147.32 77.978))
     (stroke (width 0) (type default) (color 0 0 0 0))
@@
     (stroke (width 0) (type default) (color 0 0 0 0))
   )
-  (wire (pts (xy 67.31 113.284) (xy 58.928 113.284))
+  (wire (pts (xy 66.294 113.284) (xy 58.928 113.284))
     (stroke (width 0) (type default) (color 0 0 0 0))
   )
@@
     (stroke (width 0) (type default) (color 0 0 0 0))
   )
-  (wire (pts (xy 98.552 116.078) (xy 67.31 116.078))
+  (wire (pts (xy 98.552 116.078) (xy 66.294 116.078))
     (stroke (width 0) (type default) (color 0 0 0 0))
   )
@@
     (stroke (width 0) (type default) (color 0 0 0 0))
   )
+  (wire (pts (xy 73.66 100.838) (xy 84.836 100.838))
+    (stroke (width 0) (type default) (color 0 0 0 0))
+  )
   (wire (pts (xy 147.32 77.978) (xy 147.32 76.708))
     (stroke (width 0) (type default) (color 0 0 0 0))
@@
     (stroke (width 0) (type default) (color 0 0 0 0))
   )
-  (wire (pts (xy 67.31 108.966) (xy 58.928 108.966))
+  (wire (pts (xy 68.072 108.966) (xy 58.928 108.966))
     (stroke (width 0) (type default) (color 0 0 0 0))
   )
@@
     (stroke (width 0) (type default) (color 0 0 0 0))
   )
+  (wire (pts (xy 92.456 100.838) (xy 98.552 100.838))
+    (stroke (width 0) (type default) (color 0 0 0 0))
+  )
   (wire (pts (xy 188.214 117.602) (xy 188.214 123.698))
     (stroke (width 0) (type default) (color 0 0 0 0))
@@
     (stroke (width 0) (type default) (color 0 0 0 0))
   )
+  (wire (pts (xy 67.818 100.838) (xy 73.66 100.838))
+    (stroke (width 0) (type default) (color 0 0 0 0))
+  )
   (wire (pts (xy 134.112 133.858) (xy 152.908 133.858))
     (stroke (width 0) (type default) (color 0 0 0 0))
@@
     (stroke (width 0) (type default) (color 0 0 0 0))
   )
-  (wire (pts (xy 67.31 110.998) (xy 67.31 108.966))
+  (wire (pts (xy 68.072 113.284) (xy 68.072 108.966))
     (stroke (width 0) (type default) (color 0 0 0 0))
   )
@@
     (stroke (width 0) (type default) (color 0 0 0 0))
   )
+  (wire (pts (xy 86.614 110.998) (xy 86.614 113.284))
+    (stroke (width 0) (type default) (color 0 0 0 0))
+  )
   (wire (pts (xy 59.69 98.298) (xy 98.552 98.298))
     (stroke (width 0) (type default) (color 0 0 0 0))
@@
     (stroke (width 0) (type default) (color 0 0 0 0))
   )
-  (wire (pts (xy 67.31 116.078) (xy 67.31 113.284))
+  (wire (pts (xy 66.294 116.078) (xy 66.294 113.284))
     (stroke (width 0) (type default) (color 0 0 0 0))
   )
@@
     (stroke (width 0) (type default) (color 0 0 0 0))
   )
+  (wire (pts (xy 98.552 110.998) (xy 86.614 110.998))
+    (stroke (width 0) (type default) (color 0 0 0 0))
+  )
   (wire (pts (xy 96.52 74.422) (xy 28.956 74.422))
     (stroke (width 0) (type default) (color 0 0 0 0))
@@
     (stroke (width 0) (type default) (color 0 0 0 0))
   )
+  (wire (pts (xy 56.642 100.838) (xy 67.818 100.838))
+    (stroke (width 0) (type default) (color 0 0 0 0))
+  )
   (wire (pts (xy 98.552 88.138) (xy 98.552 86.106))
     (stroke (width 0) (type default) (color 0 0 0 0))
@@
     (stroke (width 0) (type default) (color 0 0 0 0))
   )
+  (wire (pts (xy 68.072 113.284) (xy 86.614 113.284))
+    (stroke (width 0) (type default) (color 0 0 0 0))
+  )
   (wire (pts (xy 93.218 73.152) (xy 19.05 73.152))
     (stroke (width 0) (type default) (color 0 0 0 0))
@@
   (wire (pts (xy 98.552 86.106) (xy 58.674 86.106))
     (stroke (width 0) (type default) (color 0 0 0 0))
+  )
+  (text "Note 1 - populate either R88 or R89. If U5 pin 51\nis programmed to go low after boot, populate R89.\nOtherwise populate R88."
+    (at 18.542 165.862 0)
+    (effects (font (size 1.27 1.27)) (justify left bottom))
   )
   (global_label "+3.3V" (shape input) (at 189.23 34.29 90) (fields_autoplaced)
@@
     (effects (font (size 1.27 1.27)) (justify right))
     (property "Intersheet References" "${INTERSHEET_REFS}" (id 0) (at 193.3241 126.4126 0)
+      (effects (font (size 1.27 1.27)) (justify right) hide)
+    )
+  )
+  (global_label "buffer_enable" (shape output) (at 56.642 100.838 180) (fields_autoplaced)
+    (effects (font (size 1.27 1.27)) (justify right))
+    (property "Intersheet References" "${INTERSHEET_REFS}" (id 0) (at 41.3475 100.7586 0)
       (effects (font (size 1.27 1.27)) (justify right) hide)
     )
@@
   (symbol (lib_id "Connector:TestPoint") (at 80.264 103.378 90) (unit 1)
     (in_bom yes) (on_board yes)
-    (property "Reference" "TP12" (id 0) (at 73.914 103.378 90))
+    (property "Reference" "TP12" (id 0) (at 80.518 104.648 90))
     (property "Value" "test" (id 1) (at 82.55 102.108 90)
       (effects (font (size 1.27 1.27)) hide)
@@
     (pin "1")
     (pin "2")
+  )
+  (symbol (lib_id "Connector:TestPoint") (at 67.818 100.838 180) (unit 1)
+    (in_bom yes) (on_board yes)
+    (property "Reference" "TP23" (id 0) (at 63.754 102.362 0))
+    (property "Value" "test" (id 1) (at 66.548 98.552 90)
+      (effects (font (size 1.27 1.27)) hide)
+    )
+    (property "Footprint" "Connector_PinHeader_1.00mm:PinHeader_1x01_P1.00mm_Vertical" (id 2) (at 62.738 100.838 0)
+      (effects (font (size 1.27 1.27)) hide)
+    )
+    (property "Datasheet" "~" (id 3) (at 62.738 100.838 0)
+      (effects (font (size 1.27 1.27)) hide)
+    )
+    (pin "1")
   )
   (symbol (lib_id "power:GND") (at 31.75 70.358 90) (mirror x) (unit 1)
@@
     (pin "1")
   )
+  (symbol (lib_id "power:GND") (at 73.66 108.458 0) (unit 1)
+    (in_bom yes) (on_board yes)
+    (property "Reference" "#PWR01" (id 0) (at 73.66 114.808 0)
+      (effects (font (size 1.27 1.27)) hide)
+    )
+    (property "Value" "GND" (id 1) (at 76.962 108.712 0))
+    (property "Footprint" "" (id 2) (at 73.66 108.458 0)
+      (effects (font (size 1.27 1.27)) hide)
+    )
+    (property "Datasheet" "" (id 3) (at 73.66 108.458 0)
+      (effects (font (size 1.27 1.27)) hide)
+    )
+    (pin "1")
+  )
   (symbol (lib_id "Device:C") (at 164.592 133.858 90) (unit 1)
     (in_bom yes) (on_board yes)
@@
     (pin "2")
   )
+  (symbol (lib_id "Device:R_US") (at 88.646 100.838 90) (unit 1)
+    (in_bom yes) (on_board yes)
+    (property "Reference" "R89" (id 0) (at 92.71 102.108 90))
+    (property "Value" "0" (id 1) (at 85.852 101.854 90))
+    (property "Footprint" "Resistor_SMD:R_0805_2012Metric_Pad1.20x1.40mm_HandSolder" (id 2) (at 88.9 99.822 90)
+      (effects (font (size 1.27 1.27)) hide)
+    )
+    (property "Datasheet" "~" (id 3) (at 88.646 100.838 0)
+      (effects (font (size 1.27 1.27)) hide)
+    )
+    (property "Model" "RC0805JR-070RL" (id 4) (at 88.646 100.838 0)
+      (effects (font (size 1.27 1.27)) hide)
+    )
+    (pin "1")
+    (pin "2")
+  )
   (symbol (lib_id "Device:R_US") (at 208.026 126.492 90) (unit 1)
     (in_bom yes) (on_board yes)
@@
       (effects (font (size 1.27 1.27)) hide)
     )
+    (pin "1")
+    (pin "2")
+  )
+  (symbol (lib_id "Device:R_US") (at 73.66 104.648 180) (unit 1)
+    (in_bom yes) (on_board yes)
+    (property "Reference" "R88" (id 0) (at 70.866 105.918 90))
+    (property "Value" "0" (id 1) (at 74.676 107.442 90))
+    (property "Footprint" "Resistor_SMD:R_0805_2012Metric_Pad1.20x1.40mm_HandSolder" (id 2) (at 72.644 104.394 90)
+      (effects (font (size 1.27 1.27)) hide)
+    )
+    (property "Datasheet" "~" (id 3) (at 73.66 104.648 0)
+      (effects (font (size 1.27 1.27)) hide)
+    )
+    (property "Model" "RC0805JR-070RL" (id 4) (at 73.66 104.648 0)
+      (effects (font (size 1.27 1.27)) hide)
+    )

Commit message: updating recent work
Parts:
- D11, D12, D13, D14, D15, D16, D17, D18, D19, D20: Model RB521S30T1G -> CDBW46-G
Changed lines of the file:
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@@
       (effects (font (size 1.524 1.524)) hide)
     )
-    (property "Model" "RB521S30T1G" (id 4) (at 168.402 105.918 0)
+    (property "Model" "CDBW46-G" (id 4) (at 168.402 105.918 0)
       (effects (font (size 1.27 1.27)) hide)
     )
@@
       (effects (font (size 1.524 1.524)) hide)
     )
-    (property "Model" "RB521S30T1G" (id 4) (at 186.69 103.378 0)
+    (property "Model" "CDBW46-G" (id 4) (at 186.69 103.378 0)
       (effects (font (size 1.27 1.27)) hide)
     )
@@
       (effects (font (size 1.524 1.524)) hide)
     )
-    (property "Model" "RB521S30T1G" (id 4) (at 67.056 105.918 0)
+    (property "Model" "CDBW46-G" (id 4) (at 67.056 105.918 0)
       (effects (font (size 1.27 1.27)) hide)
     )
@@
       (effects (font (size 1.524 1.524)) hide)
     )
-    (property "Model" "RB521S30T1G" (id 4) (at 168.91 90.678 0)
+    (property "Model" "CDBW46-G" (id 4) (at 168.91 90.678 0)
       (effects (font (size 1.27 1.27)) hide)
     )
@@
       (effects (font (size 1.524 1.524)) hide)
     )
-    (property "Model" "RB521S30T1G" (id 4) (at 186.69 93.218 0)
+    (property "Model" "CDBW46-G" (id 4) (at 186.69 93.218 0)
       (effects (font (size 1.27 1.27)) hide)
     )
@@
       (effects (font (size 1.524 1.524)) hide)
     )
-    (property "Model" "RB521S30T1G" (id 4) (at 168.402 100.838 0)
+    (property "Model" "CDBW46-G" (id 4) (at 168.402 100.838 0)
       (effects (font (size 1.27 1.27)) hide)
     )
@@
       (effects (font (size 1.524 1.524)) hide)
     )
-    (property "Model" "RB521S30T1G" (id 4) (at 186.436 88.138 0)
+    (property "Model" "CDBW46-G" (id 4) (at 186.436 88.138 0)
       (effects (font (size 1.27 1.27)) hide)
     )
@@
       (effects (font (size 1.524 1.524)) hide)
     )
-    (property "Model" "RB521S30T1G" (id 4) (at 168.91 95.758 0)
+    (property "Model" "CDBW46-G" (id 4) (at 168.91 95.758 0)
       (effects (font (size 1.27 1.27)) hide)
     )
@@
       (effects (font (size 1.524 1.524)) hide)
     )
-    (property "Model" "RB521S30T1G" (id 4) (at 66.802 95.758 0)
+    (property "Model" "CDBW46-G" (id 4) (at 66.802 95.758 0)
       (effects (font (size 1.27 1.27)) hide)
     )
@@
       (effects (font (size 1.524 1.524)) hide)
     )
-    (property "Model" "RB521S30T1G" (id 4) (at 186.69 98.298 0)
-      (effects (font (size 1.27 1.27)) hide)
-    )
+    (property "Model" "CDBW46-G" (id 4) (at 186.69 98.298 0)
+      (effects (font (size 1.27 1.27)) hide)
+    )

Commit message: corrections after first KiCad build
Parts:
- removed R88, R89: 0, Resistor_SMD:R_0805_2012Metric_Pad1.20x1.40mm_HandSolder, symbol Device:R_US
- removed TP23: test, Connector_PinHeader_1.00mm:PinHeader_1x01_P1.00mm_Vertical, symbol Connector:TestPoint
- added J15: Conn_01x03, Connector_PinHeader_2.54mm:PinHeader_1x03_P2.54mm_Vertical, symbol Connector_Generic:Conn_01x03
- TP12: footprint Connector_PinHeader_1.00mm:PinHeader_1x01_P1.00mm_Vertical -> Project_Footprints_Library:test_point
Connections:
- net GND: now also J15.3 (Pin_3)
- net buffer_enable: now also J15.2 (Pin_2)
- net pdi: now also U3.56 (PDI_DATA); no longer U3.57 (~{RESET}/PDI_CLK)
- net reset: now also U3.57 (~{RESET}/PDI_CLK); no longer U3.56 (PDI_DATA)
- net at U3.51 (PF5): now also J15.1 (Pin_1)
Other:
- moved on the sheet: TP12

Commit message: put all schematics on 50 mil grid
Other:
- moved on the sheet: C30, C32, C34, C35, C36, C37, C69, C70, D11, D12, D13, D14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

Commit message: minor corrections in prep for new build
Connections:
- net drv_fault: now also R38.2
- net at R39.2, U3.50 (PF4): no longer R38.2
- net 3to5_17/in renamed spin_pwm_3
Other:
- removed sheet 3to5_17
- moved on the sheet: R38, R39
Changed lines of the file:
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@@
   (junction (at 67.945 17.78) (diameter 0) (color 0 0 0 0)
   )
-  (junction (at 56.515 98.425) (diameter 0) (color 0 0 0 0)
-  )
   (junction (at 77.47 25.4) (diameter 0) (color 0 0 0 0)
   )
@@
   )
   (junction (at 166.37 129.54) (diameter 0) (color 0 0 0 0)
+  )
+  (junction (at 66.04 99.06) (diameter 0) (color 0 0 0 0)
   )
   (junction (at 106.68 17.78) (diameter 0) (color 0 0 0 0)
@@
     (stroke (width 0) (type default) (color 0 0 0 0))
   )
+  (wire (pts (xy 66.04 95.25) (xy 66.04 99.06))
+    (stroke (width 0) (type default) (color 0 0 0 0))
+  )
   (wire (pts (xy 137.795 101.6) (xy 134.62 101.6))
     (stroke (width 0) (type default) (color 0 0 0 0))
@@
     (stroke (width 0) (type default) (color 0 0 0 0))
   )
-  (wire (pts (xy 46.355 98.425) (xy 48.895 98.425))
-    (stroke (width 0) (type default) (color 0 0 0 0))
-  )
   (wire (pts (xy 134.62 129.54) (xy 158.115 129.54))
     (stroke (width 0) (type default) (color 0 0 0 0))
   )
+  (wire (pts (xy 66.04 99.06) (xy 67.31 99.06))
+    (stroke (width 0) (type default) (color 0 0 0 0))
+  )
   (wire (pts (xy 99.06 129.54) (xy 69.85 129.54))
     (stroke (width 0) (type default) (color 0 0 0 0))
@@
     (stroke (width 0) (type default) (color 0 0 0 0))
   )
-  (wire (pts (xy 64.77 101.6) (xy 74.295 101.6))
+  (wire (pts (xy 54.61 101.6) (xy 74.295 101.6))
     (stroke (width 0) (type default) (color 0 0 0 0))
   )
@@
     (stroke (width 0) (type default) (color 0 0 0 0))
   )
+  (wire (pts (xy 63.5 95.25) (xy 66.04 95.25))
+    (stroke (width 0) (type default) (color 0 0 0 0))
+  )
   (wire (pts (xy 116.84 58.42) (xy 119.38 58.42))
     (stroke (width 0) (type default) (color 0 0 0 0))
@@
     (stroke (width 0) (type default) (color 0 0 0 0))
   )
+  (wire (pts (xy 63.5 99.06) (xy 66.04 99.06))
+    (stroke (width 0) (type default) (color 0 0 0 0))
+  )
   (wire (pts (xy 134.62 134.62) (xy 148.59 134.62))
     (stroke (width 0) (type default) (color 0 0 0 0))
@@
     (stroke (width 0) (type default) (color 0 0 0 0))
   )
-  (wire (pts (xy 43.815 95.25) (xy 48.895 95.25))
-    (stroke (width 0) (type default) (color 0 0 0 0))
-  )
   (wire (pts (xy 58.42 25.4) (xy 67.945 25.4))
     (stroke (width 0) (type default) (color 0 0 0 0))
@@
     (stroke (width 0) (type default) (color 0 0 0 0))
   )
-  (wire (pts (xy 56.515 99.06) (xy 56.515 98.425))
-    (stroke (width 0) (type default) (color 0 0 0 0))
-  )
   (wire (pts (xy 91.44 104.14) (xy 99.06 104.14))
     (stroke (width 0) (type default) (color 0 0 0 0))
@@
     (stroke (width 0) (type default) (color 0 0 0 0))
   )
-  (wire (pts (xy 56.515 95.25) (xy 56.515 98.425))
-    (stroke (width 0) (type default) (color 0 0 0 0))
-  )
   (wire (pts (xy 99.06 139.7) (xy 97.79 139.7))
     (stroke (width 0) (type default) (color 0 0 0 0))
@@
     (stroke (width 0) (type default) (color 0 0 0 0))
   )
-  (wire (pts (xy 76.2 133.985) (xy 78.105 133.985))
-    (stroke (width 0) (type default) (color 0 0 0 0))
-  )
   (wire (pts (xy 146.685 101.6) (xy 145.415 101.6))
     (stroke (width 0) (type default) (color 0 0 0 0))
@@
     (stroke (width 0) (type default) (color 0 0 0 0))
   )
-  (wire (pts (xy 99.06 99.06) (xy 56.515 99.06))
-    (stroke (width 0) (type default) (color 0 0 0 0))
-  )
   (wire (pts (xy 134.62 78.74) (xy 149.225 78.74))
     (stroke (width 0) (type default) (color 0 0 0 0))
@@
   )
   (wire (pts (xy 145.415 96.52) (xy 146.685 96.52))
+    (stroke (width 0) (type default) (color 0 0 0 0))
+  )
+  (wire (pts (xy 74.93 99.06) (xy 99.06 99.06))
     (stroke (width 0) (type default) (color 0 0 0 0))
   )
@@
     )
   )
-  (global_label "buffer_enable" (shape output) (at 64.77 101.6 180) (fields_autoplaced)
-    (effects (font (size 1.27 1.27)) (justify right))
-    (property "Intersheet References" "${INTERSHEET_REFS}" (id 0) (at 49.4755 101.5206 0)
+  (global_label "buffer_enable" (shape output) (at 54.61 101.6 180) (fields_autoplaced)
+    (effects (font (size 1.27 1.27)) (justify right))
+    (property "Intersheet References" "${INTERSHEET_REFS}" (id 0) (at 39.3155 101.5206 0)
       (effects (font (size 1.27 1.27)) (justify right) hide)
     )
   )
-  (global_label "+3.3V" (shape input) (at 43.815 95.25 180) (fields_autoplaced)
-    (effects (font (size 1.27 1.27)) (justify right))
-    (property "Intersheet References" "${INTERSHEET_REFS}" (id 0) (at 35.7171 95.1706 0)
+  (global_label "+3.3V" (shape input) (at 55.88 95.25 180) (fields_autoplaced)
+    (effects (font (size 1.27 1.27)) (justify right))
+    (property "Intersheet References" "${INTERSHEET_REFS}" (id 0) (at 47.7821 95.1706 0)
       (effects (font (size 1.27 1.27)) (justify right) hide)
     )
@@
     )
   )
-  (hierarchical_label "spin_pwm" (shape output) (at 76.2 133.985 180)
+  (hierarchical_label "spin_pwm_3" (shape output) (at 90.805 134.62 180)
     (effects (font (size 1.27 1.27)) (justify right))
   )
@@
     (effects (font (size 1.27 1.27)) (justify right))
   )
-  (hierarchical_label "drv_fault" (shape input) (at 46.355 98.425 180)
+  (hierarchical_label "drv_fault" (shape input) (at 63.5 99.06 180)
     (effects (font (size 1.27 1.27)) (justify right))
   )
@@
     (pin "2")
   )
-  (symbol (lib_id "Device:R_US") (at 52.705 95.25 90) (unit 1)
-    (in_bom yes) (on_board yes)
-    (property "Reference" "R38" (id 0) (at 52.705 93.345 90))
-    (property "Value" "2.4k" (id 1) (at 48.133 93.726 90))
-    (property "Footprint" "Resistor_SMD:R_0805_2012Metric_Pad1.20x1.40mm_HandSolder" (id 2) (at 52.959 94.234 90)
-      (effects (font (size 1.27 1.27)) hide)
-    )
-    (property "Datasheet" "~" (id 3) (at 52.705 95.25 0)
-      (effects (font (size 1.27 1.27)) hide)
-    )
-    (property "Model" "RC0805JR-072K4L" (id 4) (at 52.705 95.25 0)
+  (symbol (lib_id "Device:R_US") (at 59.69 95.25 90) (unit 1)
+    (in_bom yes) (on_board yes)
+    (property "Reference" "R38" (id 0) (at 59.69 93.345 90))
+    (property "Value" "2.4k" (id 1) (at 59.69 91.44 90))
+    (property "Footprint" "Resistor_SMD:R_0805_2012Metric_Pad1.20x1.40mm_HandSolder" (id 2) (at 59.944 94.234 90)
+      (effects (font (size 1.27 1.27)) hide)
+    )
+    (property "Datasheet" "~" (id 3) (at 59.69 95.25 0)
+      (effects (font (size 1.27 1.27)) hide)
+    )
+    (property "Model" "RC0805JR-072K4L" (id 4) (at 59.69 95.25 0)
       (effects (font (size 1.27 1.27)) hide)
     )
@@
     (pin "3")
   )
-  (symbol (lib_id "Device:R_US") (at 52.705 98.425 90) (unit 1)
-    (in_bom yes) (on_board yes)
-    (property "Reference" "R39" (id 0) (at 48.895 99.695 90))
-    (property "Value" "180" (id 1) (at 48.133 96.901 90))
-    (property "Footprint" "Resistor_SMD:R_0805_2012Metric_Pad1.20x1.40mm_HandSolder" (id 2) (at 52.959 97.409 90)
-      (effects (font (size 1.27 1.27)) hide)
-    )
-    (property "Datasheet" "~" (id 3) (at 52.705 98.425 0)
-      (effects (font (size 1.27 1.27)) hide)
-    )
-    (property "Model" "RMCF0805JT180R" (id 4) (at 52.705 98.425 0)
+  (symbol (lib_id "Device:R_US") (at 71.12 99.06 90) (unit 1)
+    (in_bom yes) (on_board yes)
+    (property "Reference" "R39" (id 0) (at 77.47 97.79 90))
+    (property "Value" "180" (id 1) (at 70.485 96.52 90))
+    (property "Footprint" "Resistor_SMD:R_0805_2012Metric_Pad1.20x1.40mm_HandSolder" (id 2) (at 71.374 98.044 90)
+      (effects (font (size 1.27 1.27)) hide)
+    )
+    (property "Datasheet" "~" (id 3) (at 71.12 99.06 0)
+      (effects (font (size 1.27 1.27)) hide)
+    )
+    (property "Model" "RMCF0805JT180R" (id 4) (at 71.12 99.06 0)
       (effects (font (size 1.27 1.27)) hide)
     )
@@
       (effects (font (size 1.27 1.27)) (justify left))
     )
-  )
-  (sheet (at 78.105 132.08) (size 12.7 3.81)
-    (stroke (width 0.1524) (type solid) (color 0 0 0 0))
-    (fill (color 0 0 0 0.0000))
-    (property "Sheet name" "3to5_17" (id 0) (at 91.313 134.112 0)
-      (effects (font (size 1.27 1.27)) (justify left bottom))
-    )
-    (property "Sheet file" "level_shifter.kicad_sch" (id 1) (at 78.105 136.4746 0)
-      (effects (font (size 1.27 1.27)) (justify left top) hide)
-    )
-    (pin "in" input (at 90.805 134.62 0)
-      (effects (font (size 1.27 1.27)) (justify right))
-    )
-    (pin "out" output (at 78.105 133.985 180)
-      (effects (font (size 1.27 1.27)) (justify left))
-    )
