File: microprocessor.kicad_sch (KiCad schematic)
At the start: 37 parts, among them J15 Conn_01x03, J4 Conn_02x03_Odd_Even, U3 ATxmega192A3U-A, X1 ABLS-16.000MHZ-B4-T

Commit message: first commit of V18
Parts:
- removed D11, D12, D13, D14, D15, D16, D17, D18, D19, D20: CDBW46-G, Project_Footprints_Library:CDBW46-G, symbol 1LibBBCTRL:CDBW46-G
- removed R38: 2.4k, Resistor_SMD:R_0805_2012Metric_Pad1.20x1.40mm_HandSolder, symbol Device:R_US
- removed R39: 180, Resistor_SMD:R_0805_2012Metric_Pad1.20x1.40mm_HandSolder, symbol Device:R_US
- removed TP12: test, Project_Footprints_Library:test_point, symbol Connector:TestPoint
- added R7: 10k, Resistor_SMD:R_0805_2012Metric_Pad1.20x1.40mm_HandSolder, symbol Device:R_US
- added TP19: AVR_TP, Project_Footprints_Library:test_point, symbol Connector:TestPoint
Connections:
- net 3to5_10/in is gone; now on net dir_3: U3.43 (PE7)
- net 3to5_12/in is gone; now on net out_1: U3.31 (PD5)
- net 3to5_13/in is gone; now on net out_2: U3.41 (PE5)
- net 3to5_14/in is gone; now on net out_15: U3.3 (PA5)
- net 3to5_15/in is gone; now on net out_16: U3.2 (PA4)
- net 3to5_16/in is gone; now on net out_21: U3.48 (PF2)
- net 3to5_3/in is gone; now on net step_0: U3.26 (PD0)
- net 3to5_4/in is gone; now on net step_1: U3.36 (PE0)
- net 3to5_5/in is gone; now on net step_2: U3.46 (PF0)
- net 3to5_6/in is gone; now on net step_3: U3.40 (PE4)
- net 3to5_7/in is gone; now on net dir_0: U3.38 (PE2)
- net 3to5_8/in is gone; now on net dir_1: U3.39 (PE3)
- net 3to5_9/in is gone; now on net dir_2: U3.42 (PE6)
- net +3.3V: now also R7.1
- net in_10: now also U3.13 (PB7)
- net in_11: now also U3.8 (PB2)
- net in_12: now also U3.9 (PB3)
- net in_22: now also U3.55 (PF7)
- net in_23: now also U3.49 (PF3)
- net in_3: now also U3.6 (AREFB/PB0)
- net in_4: now also U3.7 (PB1)
- net in_5: now also U3.10 (PB4)
- net in_8: now also U3.11 (PB5)
- net in_9: now also U3.12 (PB6)
- net nSLEEP: now reaches U3.54 (PF6)
- net at U3.50 (PF4): now also R7.2, TP19.1
- net stall_0 renamed nFAULT_0
- net stall_1 renamed nFAULT_1
- net stall_2 renamed nFAULT_2
- net stall_3 renamed nFAULT_3
Other:
- removed sheet 3to5_10
- removed sheet 3to5_12
- removed sheet 3to5_13
- removed sheet 3to5_14
- removed sheet 3to5_15
- removed sheet 3to5_16
- removed sheet 3to5_3
- removed sheet 3to5_4
- removed sheet 3to5_5
- removed sheet 3to5_6
- removed sheet 3to5_7
- removed sheet 3to5_8
- removed sheet 3to5_9

Commit message: added pull-up to buffer_enable
Parts:
- added R46: 10k, Resistor_SMD:R_0805_2012Metric_Pad1.20x1.40mm_HandSolder, symbol Device:R_US
Connections:
- net +3.3V: now also R46.2
- net buffer_enable: now also R46.1
Changed lines of the file:
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@@
   (junction (at 173.355 124.46) (diameter 0) (color 0 0 0 0)
+  )
+  (junction (at 57.15 101.6) (diameter 0) (color 0 0 0 0)
   )
   (junction (at 166.37 129.54) (diameter 0) (color 0 0 0 0)
@@
     (stroke (width 0) (type default) (color 0 0 0 0))
   )
+  (wire (pts (xy 57.15 101.6) (xy 74.295 101.6))
+    (stroke (width 0) (type default) (color 0 0 0 0))
+  )
   (wire (pts (xy 31.75 116.84) (xy 25.4 116.84))
     (stroke (width 0) (type default) (color 0 0 0 0))
@@
     (stroke (width 0) (type default) (color 0 0 0 0))
   )
-  (wire (pts (xy 54.61 101.6) (xy 74.295 101.6))
+  (wire (pts (xy 54.61 101.6) (xy 57.15 101.6))
     (stroke (width 0) (type default) (color 0 0 0 0))
   )
@@
     (property "Intersheet References" "${INTERSHEET_REFS}" (id 0) (at 63.0221 98.9806 0)
       (effects (font (size 1.27 1.27)) (justify right) hide)
+    )
+  )
+  (global_label "+3.3V" (shape input) (at 57.15 93.98 90) (fields_autoplaced)
+    (effects (font (size 1.27 1.27)) (justify left))
+    (property "Intersheet References" "${INTERSHEET_REFS}" (id 0) (at 57.2294 85.8821 90)
+      (effects (font (size 1.27 1.27)) (justify left) hide)
     )
   )
@@
       (effects (font (size 1.27 1.27)) hide)
     )
+    (pin "1")
+    (pin "2")
+  )
+  (symbol (lib_id "Device:R_US") (at 57.15 97.79 180) (unit 1)
+    (in_bom yes) (on_board yes)
+    (property "Reference" "R46" (id 0) (at 55.118 93.218 90))
+    (property "Value" "10k" (id 1) (at 55.0981 97.79 90))
+    (property "Footprint" "Resistor_SMD:R_0805_2012Metric_Pad1.20x1.40mm_HandSolder" (id 2) (at 56.134 97.536 90)
+      (effects (font (size 1.27 1.27)) hide)
+    )
+    (property "Datasheet" "~" (id 3) (at 57.15 97.79 0)
+      (effects (font (size 1.27 1.27)) hide)
+    )
+    (property "Model" "RC0805FR-0710KL" (id 4) (at 57.15 97.79 0)
+      (effects (font (size 1.27 1.27)) hide)
+    )

Commit message: added some testpoints
Parts:
- added TP27, TP29: CS1, Project_Footprints_Library:test_point, symbol Connector:TestPoint
- added TP28: CS2, Project_Footprints_Library:test_point, symbol Connector:TestPoint
- added TP30: CS0, Project_Footprints_Library:test_point, symbol Connector:TestPoint
- added TP31: sck, Project_Footprints_Library:test_point, symbol Connector:TestPoint
- added TP32: mosi, Project_Footprints_Library:test_point, symbol Connector:TestPoint
- added TP33: miso, Project_Footprints_Library:test_point, symbol Connector:TestPoint
- U3: value ATxmega192A3U-A -> ATXMEGA256A3U-AU; Model ATxmega192A3U-A -> ATXMEGA256A3U-AU
Connections:
- net cs_0: now also TP30.1
- net cs_1: now also TP27.1
- net cs_2: now also TP28.1
- net cs_3: now also TP29.1
- net miso: now also TP33.1
- net mosi: now also TP32.1
- net sck: now also TP31.1

Commit message: Move back to drv8711
Parts:
- removed R46, R7: 10k, Resistor_SMD:R_0805_2012Metric_Pad1.20x1.40mm_HandSolder, symbol Device:R_US
- removed TP27, TP29: CS1, Project_Footprints_Library:test_point, symbol Connector:TestPoint
- removed TP28: CS2, Project_Footprints_Library:test_point, symbol Connector:TestPoint
- removed TP30: CS0, Project_Footprints_Library:test_point, symbol Connector:TestPoint
- removed TP31: sck, Project_Footprints_Library:test_point, symbol Connector:TestPoint
- removed TP32: mosi, Project_Footprints_Library:test_point, symbol Connector:TestPoint
- removed TP33: miso, Project_Footprints_Library:test_point, symbol Connector:TestPoint
- added D11, D12, D13, D14, D15, D16, D17, D18, D19, D20: CDBW46-G, Project_Footprints_Library:CDBW46-G, symbol 1LibBBCTRL:CDBW46-G
- added R38: 2.4k, Resistor_SMD:R_0805_2012Metric_Pad1.20x1.40mm_HandSolder, symbol Device:R_US
- added R39: 180, Resistor_SMD:R_0805_2012Metric_Pad1.20x1.40mm_HandSolder, symbol Device:R_US
- added R91: 10k, Resistor_SMD:R_0805_2012Metric_Pad1.20x1.40mm_HandSolder, symbol Device:R_US
- added TP12, TP16, TP17, TP18, TP20, TP21, TP22: test, Project_Footprints_Library:test_point, symbol Connector:TestPoint
- TP19: value AVR_TP -> test
- U3: value ATXMEGA256A3U-AU -> ATxmega256A3U-AU; Model ATXMEGA256A3U-AU -> ATxmega256A3U-AU
Connections:
- net +3.3V: now also R38.1, R91.1
- net buffer_enable: now also R91.2
- net cs_0: now also TP19.1
- net cs_1: now also TP16.1
- net cs_2: now also TP17.1
- net cs_3: now also TP18.1
- net dir_0: no longer U3.38 (PE2)
- net dir_1: no longer U3.39 (PE3)
- net dir_2: no longer U3.42 (PE6)
- net dir_3: no longer U3.43 (PE7)
- net in_10: now also D14.1; no longer U3.13 (PB7)
- net in_11: now also D18.1; no longer U3.8 (PB2)
- net in_12: now also D16.1; no longer U3.9 (PB3)
- net in_22: now also D12.1; no longer U3.55 (PF7)
- net in_23: now also D11.1; no longer U3.49 (PF3)
- net in_3: now also D17.1; no longer U3.6 (AREFB/PB0)
- net in_4: now also D15.1; no longer U3.7 (PB1)
- net in_5: now also D19.1; no longer U3.10 (PB4)
- net in_8: now also D13.1; no longer U3.11 (PB5)
- net in_9: now also D20.1; no longer U3.12 (PB6)
- net miso: now also TP21.1
- net mosi: now also TP20.1
- net out_1: no longer U3.31 (PD5)
- net out_15: no longer U3.3 (PA5)
- net out_16: no longer U3.2 (PA4)
- net out_2: no longer U3.41 (PE5)
- net out_21: no longer U3.48 (PF2)
- net sck: now also TP22.1
- net step_0: no longer U3.26 (PD0)
- net step_1: no longer U3.36 (PE0)
- net step_2: no longer U3.46 (PF0)
- net step_3: no longer U3.40 (PE4)
- net at U3.50 (PF4): now also R39.2; no longer TP19.1
- net nFAULT_0 renamed stall_0
- net nFAULT_1 renamed stall_1
- net nFAULT_2 renamed stall_2
- net nFAULT_3 renamed stall_3
- net nSLEEP: no longer names the net of U3.54 (PF6)
- net nSLEEP: now also TP12.1
- new net: D14.2, U3.13 (PB7)
- new net: D20.2, U3.12 (PB6)
- new net: D12.2, U3.55 (PF7)
- new net: D19.2, U3.10 (PB4)
- new net: D13.2, U3.11 (PB5)
- new net: D11.2, U3.49 (PF3)
- new net: D17.2, U3.6 (AREFB/PB0)
- new net: D15.2, U3.7 (PB1)
- new net: D18.2, U3.8 (PB2)
- new net: D16.2, U3.9 (PB3)
- new net 3to5_10/in: U3.43 (PE7)
- new net 3to5_12/in: U3.31 (PD5)
- new net 3to5_13/in: U3.41 (PE5)
- new net 3to5_14/in: U3.3 (PA5)
- new net 3to5_15/in: U3.2 (PA4)
- new net 3to5_16/in: U3.48 (PF2)
- new net 3to5_3/in: U3.26 (PD0)
- new net 3to5_4/in: U3.36 (PE0)
- new net 3to5_5/in: U3.46 (PF0)
- new net 3to5_6/in: U3.40 (PE4)
- new net 3to5_7/in: U3.38 (PE2)
- new net 3to5_8/in: U3.39 (PE3)
- new net 3to5_9/in: U3.42 (PE6)
- new net drv_fault: R38.2, R39.1
Other:
- added sheet 3to5_10 (level_shifter.kicad_sch)
- added sheet 3to5_12 (level_shifter.kicad_sch)
- added sheet 3to5_13 (level_shifter.kicad_sch)
- added sheet 3to5_14 (level_shifter.kicad_sch)
- added sheet 3to5_15 (level_shifter.kicad_sch)
- added sheet 3to5_16 (level_shifter.kicad_sch)
- added sheet 3to5_3 (level_shifter.kicad_sch)
- added sheet 3to5_4 (level_shifter.kicad_sch)
- added sheet 3to5_5 (level_shifter.kicad_sch)
- added sheet 3to5_6 (level_shifter.kicad_sch)
- added sheet 3to5_7 (level_shifter.kicad_sch)
- added sheet 3to5_8 (level_shifter.kicad_sch)
- added sheet 3to5_9 (level_shifter.kicad_sch)
- note removed: "Note 1 - populate either R88 or R89. If U5 pin 51 is programmed to go low after boot, populate R89. Otherwise populate R88."
- moved on the sheet: C70, R67

Commit message: All DRC errors cleared after conversion to Kicad V7
Other:
- moved on the sheet: C31, C32, C33, C34, C35, C69, D10, D13, D14, D15, D16, D17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

Commit message: swapped avr pins 21 and 23 (mosi and sck) to accomodate xmegaa3 chip
Connections:
- net at R67.1: now also U3.23 (PC7); no longer U3.21 (PC5)
- net at R66.1: now also U3.21 (PC5); no longer U3.23 (PC7)
Other:
- moved on the sheet: C69, C70, R66, R67, TP20, TP22

Commit message: changed mosi and sck resistors from 180 ohm to 100 ohm
Parts:
- removed R66, R67: 180, Resistor_SMD:R_0805_2012Metric_Pad1.20x1.40mm_HandSolder, symbol Device:R_US
- added R12 (x2): 100, Resistor_SMD:R_0805_2012Metric_Pad1.20x1.40mm_HandSolder, symbol Device:R_US
Connections:
- net mosi: now also R12.2
- net sck: now also R12.2
- net at U3.23 (PC7): now also R12.1
- net at U3.21 (PC5): now also R12.1
Changed lines of the file:
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@@
-    )
-  )
-  (symbol (lib_id "Device:R_US") (at 157.48 129.54 90) (unit 1)
-    (in_bom yes) (on_board yes) (dnp no)
-    (property "Reference" "R67" (at 157.48 132.08 90)
-      (effects (font (size 1.27 1.27)))
-    )
-    (property "Value" "180" (at 150.876 128.016 90)
-      (effects (font (size 1.27 1.27)))
-    )
-    (property "Footprint" "Resistor_SMD:R_0805_2012Metric_Pad1.20x1.40mm_HandSolder" (at 157.734 128.524 90)
-      (effects (font (size 1.27 1.27)) hide)
-    )
-    (property "Datasheet" "~" (at 157.48 129.54 0)
-      (effects (font (size 1.27 1.27)) hide)
-    )
-    (property "Model" "RMCF0805JT180R" (at 157.48 129.54 0)
-      (effects (font (size 1.27 1.27)) hide)
-    )
-    (pin "1")
-    (pin "2")
-    (instances
-      (project "BuildboticsController"
-        (path "/7f2164be-b8eb-4dbc-bc7c-152cd10e724f/3adf10c7-5d86-4ad9-b91c-31c97a8ff0e6"
-          (reference "R67") (unit 1)
-        )
-      )
     )
   )
@@
         (path "/7f2164be-b8eb-4dbc-bc7c-152cd10e724f/3adf10c7-5d86-4ad9-b91c-31c97a8ff0e6"
           (reference "D12") (unit 1)
-        )
-      )
-    )
-  )
-  (symbol (lib_id "Device:R_US") (at 161.29 124.46 90) (unit 1)
-    (in_bom yes) (on_board yes) (dnp no)
-    (property "Reference" "R66" (at 165.1 123.19 90)
-      (effects (font (size 1.27 1.27)))
-    )
-    (property "Value" "180" (at 157.226 125.984 90)
-      (effects (font (size 1.27 1.27)))
-    )
-    (property "Footprint" "Resistor_SMD:R_0805_2012Metric_Pad1.20x1.40mm_HandSolder" (at 161.544 123.444 90)
-      (effects (font (size 1.27 1.27)) hide)
-    )
-    (property "Datasheet" "~" (at 161.29 124.46 0)
-      (effects (font (size 1.27 1.27)) hide)
-    )
-    (property "Model" "RMCF0805JT180R" (at 161.29 124.46 0)
-      (effects (font (size 1.27 1.27)) hide)
-    )
-    (pin "1")
-    (pin "2")
-    (instances
-      (project "BuildboticsController"
-        (path "/7f2164be-b8eb-4dbc-bc7c-152cd10e724f/3adf10c7-5d86-4ad9-b91c-31c97a8ff0e6"
-          (reference "R66") (unit 1)
         )
       )
@@
       (effects (font (size 1.27 1.27)))
     )
-    (property "Value" "130pF" (at 159.766 120.65 90)
+    (property "Value" "130pF" (at 158.75 115.57 90)
       (effects (font (size 1.27 1.27)))
     )
@@
     )
   )
+  (symbol (lib_id "Device:R_US") (at 161.29 124.46 90) (unit 1)
+    (in_bom yes) (on_board yes) (dnp no)
+    (property "Reference" "R12" (at 154.94 123.19 90)
+      (effects (font (size 1.27 1.27)))
+    )
+    (property "Value" "100" (at 161.29 122.4081 90)
+      (effects (font (size 1.27 1.27)))
+    )
+    (property "Footprint" "Resistor_SMD:R_0805_2012Metric_Pad1.20x1.40mm_HandSolder" (at 161.544 123.444 90)
+      (effects (font (size 1.27 1.27)) hide)
+    )
+    (property "Datasheet" "~" (at 161.29 124.46 0)
+      (effects (font (size 1.27 1.27)) hide)
+    )
+    (property "Model" "RC0805FR-7W100RL" (at 161.29 124.46 0)
+      (effects (font (size 1.27 1.27)) hide)
+    )
+    (pin "1")
+    (pin "2")
+    (instances
+      (project "BuildboticsController"
+        (path "/7f2164be-b8eb-4dbc-bc7c-152cd10e724f/15e1e1b6-b278-4e13-8221-f9f8917bc709"
+          (reference "R12") (unit 1)
+        )
+        (path "/7f2164be-b8eb-4dbc-bc7c-152cd10e724f/3adf10c7-5d86-4ad9-b91c-31c97a8ff0e6"
+          (reference "R66") (unit 1)
+        )
+      )
+    )
+  )
   (symbol (lib_id "Device:C") (at 168.91 135.89 90) (unit 1)
     (in_bom yes) (on_board yes) (dnp no)
@@
         )
       )
+    )
+  )
+  (symbol (lib_id "Device:R_US") (at 157.48 129.54 90) (unit 1)
+    (in_bom yes) (on_board yes) (dnp no)
+    (property "Reference" "R12" (at 152.4 128.27 90)
+      (effects (font (size 1.27 1.27)))
+    )
+    (property "Value" "100" (at 161.29 128.27 90)
+      (effects (font (size 1.27 1.27)))
+    )
+    (property "Footprint" "Resistor_SMD:R_0805_2012Metric_Pad1.20x1.40mm_HandSolder" (at 157.734 128.524 90)
+      (effects (font (size 1.27 1.27)) hide)
+    )
+    (property "Datasheet" "~" (at 157.48 129.54 0)
+      (effects (font (size 1.27 1.27)) hide)
+    )
+    (property "Model" "RC0805FR-7W100RL" (at 157.48 129.54 0)
+      (effects (font (size 1.27 1.27)) hide)
+    )
+    (pin "1")
+    (pin "2")
+    (instances
+      (project "BuildboticsController"
+        (path "/7f2164be-b8eb-4dbc-bc7c-152cd10e724f/15e1e1b6-b278-4e13-8221-f9f8917bc709"
+          (reference "R12") (unit 1)
+        )
+        (path "/7f2164be-b8eb-4dbc-bc7c-152cd10e724f/3adf10c7-5d86-4ad9-b91c-31c97a8ff0e6"
+          (reference "R67") (unit 1)
+        )
+      )
