File: BuildboticsController.kicad_sch (KiCad schematic)
At the start: 0 parts

Commit message: corrections after first KiCad build
Other:
- sheet Power Supply ports: added 5V_scl, 5V_sda; removed none
- sheet Raspberry Pi ports: added 5V_scl, 5V_sda; removed none

Commit message: minor corrections in prep for new build
Other:
- sheet Microprocessor ports: added spin_pwm_3; removed spin_pwm
- sheet Peripherals ports: added spin_pwm_3; removed spin_pwm
Changed lines of the file:
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@@
-      (effects (font (size 1.27 1.27)) (justify left))
-    )
-    (pin "spin_pwm" output (at 142.24 60.96 180)
       (effects (font (size 1.27 1.27)) (justify left))
     )
@@
     )
     (pin "scl" output (at 142.24 152.4 180)
+      (effects (font (size 1.27 1.27)) (justify left))
+    )
+    (pin "spin_pwm_3" output (at 142.24 60.96 180)
       (effects (font (size 1.27 1.27)) (justify left))
     )
@@
       (effects (font (size 1.27 1.27)) (justify right))
     )
-    (pin "spin_pwm" input (at 125.73 60.96 0)
+    (pin "spin_pwm_3" input (at 125.73 60.96 0)
       (effects (font (size 1.27 1.27)) (justify right))
     )
@@
     (path "/3adf10c7-5d86-4ad9-b91c-31c97a8ff0e6/2271974a-e966-4a72-869e-f0dde9603f54" (page "23"))
     (path "/15e1e1b6-b278-4e13-8221-f9f8917bc709/0f0648da-b777-4b86-9593-c9dad3aa2b60" (page "24"))
-    (path "/3adf10c7-5d86-4ad9-b91c-31c97a8ff0e6/a9417cdc-2424-4304-aaf6-a0b0354c7ed7" (page "24"))
+    (path "/7b65f6db-5358-4955-b729-25fdf7672490/db1c02e9-6be9-4c02-93db-34d7e8ec71c4" (page "24"))
     (path "/2c50321d-3924-4dc6-91c5-3e71751f45d8" (page "25"))
   )
@@
       (reference "#PWR07") (unit 1) (value "GND") (footprint "")
     )
+    (path "/7b65f6db-5358-4955-b729-25fdf7672490/db1c02e9-6be9-4c02-93db-34d7e8ec71c4/4c1553a3-e58d-47f3-9c29-daccc8bf3ae0"
+      (reference "#PWR08") (unit 1) (value "~") (footprint "")
+    )
+    (path "/7b65f6db-5358-4955-b729-25fdf7672490/db1c02e9-6be9-4c02-93db-34d7e8ec71c4/59e00934-b1fc-4af9-a866-bdf6cd199ca1"
+      (reference "#PWR09") (unit 1) (value "~") (footprint "")
+    )
     (path "/2c7a0987-643f-4f73-bdef-a41a77343a1c/1f229479-2164-4805-9748-96b8ddabc96d"
       (reference "#PWR0101") (unit 1) (value "GND") (footprint "")
@@
       (reference "#PWR0208") (unit 1) (value "~") (footprint "")
     )
-    (path "/3adf10c7-5d86-4ad9-b91c-31c97a8ff0e6/a9417cdc-2424-4304-aaf6-a0b0354c7ed7/59e00934-b1fc-4af9-a866-bdf6cd199ca1"
-      (reference "#PWR0210") (unit 1) (value "~") (footprint "")
-    )
-    (path "/3adf10c7-5d86-4ad9-b91c-31c97a8ff0e6/a9417cdc-2424-4304-aaf6-a0b0354c7ed7/4c1553a3-e58d-47f3-9c29-daccc8bf3ae0"
-      (reference "#PWR0211") (unit 1) (value "~") (footprint "")
-    )
     (path "/7b65f6db-5358-4955-b729-25fdf7672490/77460195-0ab9-47c8-9ed0-17d1e35c1265"
       (reference "#PWR0216") (unit 1) (value "GND") (footprint "")
@@
       (reference "C91") (unit 1) (value ".1uF") (footprint "Capacitor_SMD:C_0805_2012Metric_Pad1.18x1.45mm_HandSolder")
     )
-    (path "/3adf10c7-5d86-4ad9-b91c-31c97a8ff0e6/a9417cdc-2424-4304-aaf6-a0b0354c7ed7/d6134535-6919-4a7d-8d73-79f857594e1f"
+    (path "/7b65f6db-5358-4955-b729-25fdf7672490/db1c02e9-6be9-4c02-93db-34d7e8ec71c4/d6134535-6919-4a7d-8d73-79f857594e1f"
       (reference "C92") (unit 1) (value ".1uF") (footprint "Capacitor_SMD:C_0805_2012Metric_Pad1.18x1.45mm_HandSolder")
     )
@@
       (reference "J4") (unit 1) (value "Conn_02x03_Odd_Even") (footprint "Connector_PinHeader_2.54mm:PinHeader_2x03_P2.54mm_Vertical")
     )
-    (path "/7b65f6db-5358-4955-b729-25fdf7672490/4502348f-edf2-4996-8347-ae18f11ef63c"
-      (reference "J5") (unit 1) (value "DB25_Male_MountingHoles") (footprint "Project_Footprints_Library:182025113R161")
+    (path "/7b65f6db-5358-4955-b729-25fdf7672490/c8a01ed5-a627-42a7-8035-4ea94369ce97"
+      (reference "J5") (unit 1) (value "DB25_Male") (footprint "Project_Footprints_Library:182025113R161")
     )
     (path "/7b65f6db-5358-4955-b729-25fdf7672490/5c3675dd-4606-49fc-943f-72188418e513"
@@
       (reference "U26") (unit 1) (value "SN74AHC1G125DBVR") (footprint "Project_Footprints_Library:SN74AHC1G125DBVR")
     )
-    (path "/3adf10c7-5d86-4ad9-b91c-31c97a8ff0e6/a9417cdc-2424-4304-aaf6-a0b0354c7ed7/25c47cbe-8130-4d39-8fc6-fb6d8b171f6e"
-      (reference "U28") (unit 1) (value "SN74AHC1G125DBVR") (footprint "Project_Footprints_Library:SN74AHC1G125DBVR")
+    (path "/7b65f6db-5358-4955-b729-25fdf7672490/db1c02e9-6be9-4c02-93db-34d7e8ec71c4/25c47cbe-8130-4d39-8fc6-fb6d8b171f6e"
+      (reference "U27") (unit 1) (value "SN74AHC1G125DBVR") (footprint "Project_Footprints_Library:SN74AHC1G125DBVR")
     )
     (path "/7b65f6db-5358-4955-b729-25fdf7672490/3f217030-9ef7-42d3-93fa-475443c1886a"
