File: peripherals.kicad_sch (KiCad schematic)
At the start: 36 parts, among them J5 DB25_Male, J6 Conn_02x08_Odd_Even, Q25 BC856B, U16 ISL83485IBZ, U25 BSP16T1G, U29 LM358

Commit message: first commit of V18
Parts:
- added C10, C4, C44, C5: .1uF, Capacitor_SMD:C_0805_2012Metric_Pad1.18x1.45mm_HandSolder, symbol Device:C
- added D21, D22, D23, D24: ShottkeyDiodeArray, Project_Footprints_Library:RB731UT108, symbol 1LibBBCTRL:ShottkeyDiodeArray
- added U5, U9: SN74LVC4245APWR, Project_Footprints_Library:PW24, symbol 1LibBBCTRL:SN74LVC4245APWR
Connections:
- net +3.3V: now also C10.1, C4.1, U5.23 (VCCB), U5.24 (VCCB), U9.23 (VCCB), U9.24 (VCCB)
- net +5V: now also C44.1, C5.1, U5.1 (VCCA), U9.1 (VCCA)
- net GND: now also C10.2, C4.2, C44.2, C5.2, U5.11 (GND), U5.12 (GND), U5.13 (GND), U5.2 (DIR), U9.11 (GND), U9.12 (GND), U9.13 (GND), U9.2 (DIR), U9.21 (B1)
- net dir_0: now also U5.20 (B2); no longer J6.4 (Pin_4)
- net dir_1: now also U5.18 (B4); no longer J6.6 (Pin_6)
- net dir_2: now also U5.16 (B6); no longer J6.8 (Pin_8)
- net dir_3: now also U5.14 (B8); no longer J6.10 (Pin_10)
- net in_10: now also D23.6 (A); no longer J5.10
- net in_11: now also D23.4 (A); no longer J5.11
- net in_12: now also D24.6 (A); no longer J5.12
- net in_22: now also D22.4 (A); no longer J5.22 (P22)
- net in_23: now also D23.5 (A); no longer J5.23 (P23)
- net in_3: now also D21.6 (A); no longer J5.3
- net in_4: now also D21.5 (A); no longer J5.4
- net in_5: now also D21.4 (A); no longer J5.5
- net in_8: now also D22.6 (A); no longer J5.8
- net in_9: now also D22.5 (A); no longer J5.9
- net out_1: now also U9.18 (B4); no longer J5.1
- net out_15: now also U9.16 (B6); no longer J5.15 (P15)
- net out_16: now also U9.15 (B7); no longer J5.16 (P16)
- net out_2: now also U9.17 (B5); no longer J5.2
- net out_21: now also U9.20 (B2); no longer J5.21 (P21)
- net spin_pwm_3: now also U9.19 (B3)
- net step_0: now also U5.19 (B3); no longer J6.3 (Pin_3)
- net step_1: now also U5.17 (B5); no longer J6.5 (Pin_5)
- net step_2: now also U5.15 (B7); no longer J6.7 (Pin_7)
- net step_3: now also U5.21 (B1); no longer J6.9 (Pin_9)
- net drv_enable renamed motor_enable
- net spin_pwm renamed spinpwm
- net spinpwm: now also U9.5 (A3)
- new net: D21.2 (K), J5.4
- new net: D23.3 (K), J5.11
- new net: D22.2 (K), J5.9
- new net: D23.2 (K), J5.23 (P23)
- new net: D22.3 (K), J5.22 (P22)
- new net: D23.1 (K), J5.10
- new net: D22.1 (K), J5.8
- new net: D21.1 (K), J5.3
- new net: D24.1 (K), J5.12
- new net: D21.3 (K), J5.5
- new net buffer_enable: U5.22 (*OE), U9.22 (*OE)
- new net dir0: J6.4 (Pin_4), U5.4 (A2)
- new net dir1: J6.6 (Pin_6), U5.6 (A4)
- new net dir2: J6.8 (Pin_8), U5.8 (A6)
- new net dir3: J6.10 (Pin_10), U5.10 (A8)
- new net nSLEEP: U9.14 (B8)
- new net nSLP: U9.10 (A8)
- new net out1: J5.1, U9.6 (A4)
- new net out15: J5.15 (P15), U9.8 (A6)
- new net out16: J5.16 (P16), U9.9 (A7)
- new net out2: J5.2, U9.7 (A5)
- new net out21: J5.21 (P21), U9.4 (A2)
- new net step0: J6.3 (Pin_3), U5.5 (A3)
- new net step1: J6.5 (Pin_5), U5.7 (A5)
- new net step2: J6.7 (Pin_7), U5.9 (A7)
- new net step3: J6.9 (Pin_9), U5.3 (A1)
- no-connect marks 1 -> 2
Other:
- removed sheet 3_to_5_17
- moved on the sheet: C48, C71, J6
