File: peripherals.kicad_sch (KiCad schematic)
At the start: 46 parts, among them J5 DB25_Male, J6 Conn_02x08_Odd_Even, Q25 BC856B, U16 ISL83485IBZ, U25 BSP16T1G, U29 LM358, U5 SN74LVC4245APWR, U9 SN74LVC4245APWR

Commit message: added some testpoints
Parts:
- added TP26: TP_nSLP, Project_Footprints_Library:test_point, symbol Connector:TestPoint
- TP23: footprint Connector_PinHeader_2.54mm:PinHeader_1x01_P2.54mm_Vertical -> Project_Footprints_Library:test_point
Connections:
- net nSLP: now also TP26.1
Changed lines of the file:
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@@
   (junction (at 121.92 92.71) (diameter 0) (color 0 0 0 0)
+  )
+  (junction (at 254.635 69.215) (diameter 0) (color 0 0 0 0)
   )
   (junction (at 149.225 99.695) (diameter 0) (color 0 0 0 0)
@@
     (stroke (width 0) (type default) (color 0 0 0 0))
   )
+  (wire (pts (xy 254.635 69.215) (xy 238.76 69.215))
+    (stroke (width 0) (type default) (color 0 0 0 0))
+  )
   (wire (pts (xy 82.55 53.34) (xy 82.55 52.705))
     (stroke (width 0) (type default) (color 0 0 0 0))
@@
   )
   (wire (pts (xy 246.38 137.795) (xy 259.08 137.795))
+    (stroke (width 0) (type default) (color 0 0 0 0))
+  )
+  (wire (pts (xy 267.97 69.215) (xy 254.635 69.215))
     (stroke (width 0) (type default) (color 0 0 0 0))
   )
@@
     (effects (font (size 1.27 1.27)) (justify right))
   )
-  (hierarchical_label "nSLP" (shape output) (at 238.76 69.215 0)
+  (hierarchical_label "nSLP" (shape output) (at 267.97 69.215 0)
     (effects (font (size 1.27 1.27)) (justify left))
   )
@@
       (effects (font (size 1.27 1.27)) (justify left))
     )
-    (property "Footprint" "Connector_PinHeader_2.54mm:PinHeader_1x01_P2.54mm_Vertical" (id 2) (at 146.685 92.71 0)
+    (property "Footprint" "Project_Footprints_Library:test_point" (id 2) (at 146.685 92.71 0)
       (effects (font (size 1.27 1.27)) hide)
     )
@@
     (pin "9")
   )
+  (symbol (lib_id "Connector:TestPoint") (at 254.635 69.215 0) (unit 1)
+    (in_bom yes) (on_board yes) (fields_autoplaced)
+    (property "Reference" "TP26" (id 0) (at 256.032 65.0783 0)
+      (effects (font (size 1.27 1.27)) (justify left))
+    )
+    (property "Value" "TP_nSLP" (id 1) (at 256.032 67.6152 0)
+      (effects (font (size 1.27 1.27)) (justify left))
+    )
+    (property "Footprint" "Project_Footprints_Library:test_point" (id 2) (at 259.715 69.215 0)
+      (effects (font (size 1.27 1.27)) hide)
+    )
+    (property "Datasheet" "~" (id 3) (at 259.715 69.215 0)
+      (effects (font (size 1.27 1.27)) hide)
+    )
+    (pin "1")
+  )
   (symbol (lib_id "1LibBBCTRL:ShottkeyDiodeArray") (at 242.57 135.255 0) (unit 3)

Commit message: updated some part numbers
Parts:
- J5: Model 182-025-113R161 -> DB25-PL-25
- R74, R76: Model RMCF0805JT750 -> RMCF0805JT750R
Changed lines of the file:
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@@
       (effects (font (size 1.27 1.27)) hide)
     )
-    (property "Model" "RMCF0805JT750" (id 4) (at 136.525 28.575 0)
+    (property "Model" "RMCF0805JT750R" (id 4) (at 136.525 28.575 0)
       (effects (font (size 1.27 1.27)) hide)
     )
@@
       (effects (font (size 1.27 1.27)) hide)
     )
-    (property "Model" "RMCF0805JT750" (id 4) (at 136.525 46.99 0)
+    (property "Model" "RMCF0805JT750R" (id 4) (at 136.525 46.99 0)
       (effects (font (size 1.27 1.27)) hide)
     )
@@
       (effects (font (size 1.27 1.27)) hide)
     )
-    (property "Model" "182-025-113R161" (id 4) (at 259.08 122.555 0)
-      (effects (font (size 1.27 1.27)) hide)
-    )
+    (property "Model" "DB25-PL-25" (id 4) (at 259.08 122.555 0)
+      (effects (font (size 1.27 1.27)) hide)
+    )

Commit message: Move back to drv8711
Parts:
- removed C10, C4, C44, C5: .1uF, Capacitor_SMD:C_0805_2012Metric_Pad1.18x1.45mm_HandSolder, symbol Device:C
- removed D21, D22, D23, D24: ShottkeyDiodeArray, Project_Footprints_Library:RB731UT108, symbol 1LibBBCTRL:ShottkeyDiodeArray
- removed R83: 0, Resistor_SMD:R_0805_2012Metric_Pad1.20x1.40mm_HandSolder, symbol Device:R_US
- removed TP26: TP_nSLP, Project_Footprints_Library:test_point, symbol Connector:TestPoint
- removed U5, U9: SN74LVC4245APWR, Project_Footprints_Library:PW24, symbol 1LibBBCTRL:SN74LVC4245APWR
- R74, R76: Model RMCF0805JT750R -> RMCF0805JT750
- TP23: footprint Project_Footprints_Library:test_point -> Connector_PinHeader_2.54mm:PinHeader_1x01_P2.54mm_Vertical
- U29: Model LM358 -> LM358DR2G
Connections:
- net dir0 is gone; now on net dir_0: J6.4 (Pin_4)
- net dir1 is gone; now on net dir_1: J6.6 (Pin_6)
- net dir2 is gone; now on net dir_2: J6.8 (Pin_8)
- net dir3 is gone; now on net dir_3: J6.10 (Pin_10)
- net out1 is gone; now on net out_1: J5.1
- net out15 is gone; now on net out_15: J5.15 (P15)
- net out16 is gone; now on net out_16: J5.16 (P16)
- net out2 is gone; now on net out_2: J5.2
- net out21 is gone; now on net out_21: J5.21 (P21)
- net step0 is gone; now on net step_0: J6.3 (Pin_3)
- net step1 is gone; now on net step_1: J6.5 (Pin_5)
- net step2 is gone; now on net step_2: J6.7 (Pin_7)
- net step3 is gone; now on net step_3: J6.9 (Pin_9)
- net in_10: now also J5.10
- net in_11: now also J5.11
- net in_12: now also J5.12
- net in_22: now also J5.22 (P22)
- net in_23: now also J5.23 (P23)
- net in_3: now also J5.3
- net in_4: now also J5.4
- net in_5: now also J5.5
- net in_8: now also J5.8
- net in_9: now also J5.9
- net spin_0to10: now also R82.2, U29.1
- net motor_enable renamed drv_enable
- net spinpwm renamed spin_pwm
- no-connect marks 2 -> 1
Other:
- added sheet 3_to_5_17 (level_shifter.kicad_sch)
- moved on the sheet: C48, C71, J6

Commit message: All DRC errors cleared after conversion to Kicad V7
Parts:
- removed U29: LM358, Package_SO:SOIC-8_3.9x4.9mm_P1.27mm, symbol 1LibBBCTRL:LM358
- added U29: LM358, symbol Amplifier_Operational:LM358
Connections:
- net GND: now also U29.4 (V-)
- net spin_0to10: now also U29.1
- net at C80.1, C96.1, TP23.1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: now also U29.8 (V+)
- net at C95.1, R80.2: now also U29.3 (+)
- net at R81.2, R82.1: now also U29.2 (-)
Other:
- moved on the sheet: C48, C71, C80, C81, C82, C84, C85, C86, C95, C96, J5, J6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

Commit message: changed level shifter symbol
Parts:
- U29: footprint (none) -> Package_SO:SOIC-8_3.9x4.9mm_P1.27mm
Changed lines of the file:
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@@
       (effects (font (size 1.27 1.27)) hide)
     )
-    (property "Footprint" "" (at 180.34 101.6 0)
+    (property "Footprint" "Package_SO:SOIC-8_3.9x4.9mm_P1.27mm" (at 180.34 101.6 0)
       (effects (font (size 1.27 1.27)) hide)
     )
@@
       (effects (font (size 1.27 1.27)) hide)
     )
-    (property "Footprint" "" (at 180.34 101.6 0)
+    (property "Footprint" "Package_SO:SOIC-8_3.9x4.9mm_P1.27mm" (at 180.34 101.6 0)
       (effects (font (size 1.27 1.27)) hide)
     )

Commit message: added decoupling cap to U16, fixed DRC param, and corrected resulting clearance violations
Parts:
- added C93: .1uF, Capacitor_SMD:C_0805_2012Metric_Pad1.18x1.45mm_HandSolder, symbol Device:C
Connections:
- net +3.3V: now also C93.1
- net GND: now also C93.2
Changed lines of the file:
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@@
   (junction (at 142.24 133.35) (diameter 0) (color 0 0 0 0)
+  )
+  (junction (at 128.27 24.13) (diameter 0) (color 0 0 0 0)
   )
   (junction (at 246.38 114.3) (diameter 0) (color 0 0 0 0)
@@
     (stroke (width 0) (type default))
   )
+  (wire (pts (xy 128.27 24.13) (xy 128.27 34.29))
+    (stroke (width 0) (type default))
+  )
   (wire (pts (xy 170.18 116.84) (xy 170.18 118.11))
     (stroke (width 0) (type default))
@@
   )
   (wire (pts (xy 82.55 36.83) (xy 87.63 36.83))
+    (stroke (width 0) (type default))
+  )
+  (wire (pts (xy 128.27 21.59) (xy 128.27 24.13))
     (stroke (width 0) (type default))
   )
@@
     )
   )
-  (global_label "+3.3V" (shape input) (at 128.27 34.29 90) (fields_autoplaced)
+  (global_label "+3.3V" (shape input) (at 128.27 21.59 90) (fields_autoplaced)
     (effects (font (size 1.27 1.27)) (justify left))
-    (property "Intersheetrefs" "${INTERSHEET_REFS}" (at 128.1906 26.1921 90)
+    (property "Intersheetrefs" "${INTERSHEET_REFS}" (at 128.1906 13.4921 90)
       (effects (font (size 1.27 1.27)) (justify left) hide)
     )
@@
         (path "/7f2164be-b8eb-4dbc-bc7c-152cd10e724f/7b65f6db-5358-4955-b729-25fdf7672490"
           (reference "R78") (unit 1)
+        )
+      )
+    )
+  )
+  (symbol (lib_name "GND_3") (lib_id "power:GND") (at 120.65 24.13 270) (unit 1)
+    (in_bom yes) (on_board yes) (dnp no) (fields_autoplaced)
+    (property "Reference" "#PWR010" (at 114.3 24.13 0)
+      (effects (font (size 1.27 1.27)) hide)
+    )
+    (property "Value" "GND" (at 116.84 24.13 90)
+      (effects (font (size 1.27 1.27)) (justify right))
+    )
+    (property "Footprint" "" (at 120.65 24.13 0)
+      (effects (font (size 1.27 1.27)) hide)
+    )
+    (property "Datasheet" "" (at 120.65 24.13 0)
+      (effects (font (size 1.27 1.27)) hide)
+    )
+    (pin "1")
+    (instances
+      (project "BuildboticsController"
+        (path "/7f2164be-b8eb-4dbc-bc7c-152cd10e724f/7b65f6db-5358-4955-b729-25fdf7672490"
+          (reference "#PWR010") (unit 1)
         )
       )
@@
   )
   (symbol (lib_id "1LibBBCTRL:ISL83485IBZ") (at 87.63 34.29 0) (unit 1)
-    (in_bom yes) (on_board yes) (dnp no) (fields_autoplaced)
-    (property "Reference" "U16" (at 107.95 25.0624 0)
+    (in_bom yes) (on_board yes) (dnp no)
+    (property "Reference" "U16" (at 100.33 27.94 0)
       (effects (font (size 1.524 1.524)))
     )
-    (property "Value" "ISL83485IBZ" (at 107.95 28.0558 0)
+    (property "Value" "ISL83485IBZ" (at 107.95 44.45 0)
       (effects (font (size 1.524 1.524)))
     )
@@
         )
       )
+    )
+  )
+  (symbol (lib_id "Device:C") (at 124.46 24.13 270) (unit 1)
+    (in_bom yes) (on_board yes) (dnp no)
+    (property "Reference" "C93" (at 126.492 24.638 0)
+      (effects (font (size 1.27 1.27)) (justify left))
+    )
+    (property "Value" ".1uF" (at 122.428 24.638 0)
+      (effects (font (size 1.27 1.27)) (justify left))
+    )
+    (property "Footprint" "Capacitor_SMD:C_0805_2012Metric_Pad1.18x1.45mm_HandSolder" (at 120.65 25.0952 0)
+      (effects (font (size 1.27 1.27)) hide)
+    )
+    (property "Datasheet" "~" (at 124.46 24.13 0)
+      (effects (font (size 1.27 1.27)) hide)
+    )
+    (property "Model" "C0805C104M5RACTU" (at 124.46 24.13 0)
+      (effects (font (size 1.27 1.27)) hide)
+    )
+    (pin "1")
+    (pin "2")
+    (instances
+      (project "BuildboticsController"
+        (path "/7f2164be-b8eb-4dbc-bc7c-152cd10e724f/7b65f6db-5358-4955-b729-25fdf7672490"
+          (reference "C93") (unit 1)
+        )
+      )

Commit message: changed 12V supply for 0-10V out to LDO voltage regulator
Parts:
- removed C80: 1u, Capacitor_SMD:C_0805_2012Metric_Pad1.18x1.45mm_HandSolder, symbol Device:C
- removed Q25: BC856B, Project_Footprints_Library:BC856B_215, symbol 1LibBBCTRL:BC856B
- removed R88: 56k, Resistor_SMD:R_0805_2012Metric_Pad1.20x1.40mm_HandSolder, symbol Device:R_US
- removed R89: 62, Resistor_SMD:R_0805_2012Metric_Pad1.20x1.40mm_HandSolder, symbol Device:R_US
- removed U25: BSP16T1G, Project_Footprints_Library:BSP16T1G, symbol 1LibBBCTRL:BSP16T1G
- removed Z3: 12V, Package_TO_SOT_SMD:SOT-23, symbol 1LibBBCTRL:MMBZ5242BLT3G
- added C20: 1uF 100V, Capacitor_SMD:C_0805_2012Metric_Pad1.18x1.45mm_HandSolder, symbol Device:C
- added C98: 10uF, Capacitor_SMD:C_1206_3216Metric_Pad1.33x1.80mm_HandSolder, symbol Device:C
- added U25: ZXTR2012Z-7, Project_Footprints_Library:ZXTR2012Z7, symbol 1LibBBCTRL:ZXTR2012Z-7
Connections:
- net GND: now also C20.2, C98.2, U25.1 (GND)
- net Vs: now also C20.1, U25.2 (VIN_1), U25.4 (VIN_2)
- net at C96.1, TP23.1, U29.8 (V+): now also C98.1, U25.3 (VOUT)
Other:
- moved on the sheet: J6
