File: PowerSupply.kicad_sch (KiCad schematic)
At the start: 84 parts, among them J14 PROG, J2 39-30-0060, J3 ENABLE, Q10 FDC5614P, Q5 BSC040N08NS5ATMA1, Q6 BSC040N08NS5ATMA1, Q7 2N7002K, Q8 NTD5867NLT4G, Q9 2N7002K, U2 ATtiny1616-S, U4 TSC2012IDT, U6 L7987, U7 AZ1117IH-3.3TRG1, U8 LM74800QDRRRQ1

Commit message: removed autosave file and corrected schematic electrical rules check warnings and errors
Connections:
- now unconnected: U8.13 (PAD)
Changed lines of the file:
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@@
     (pin "2")
+  )
+  (symbol (lib_id "power:GND") (at 187.706 30.48 270) (unit 1)
+    (in_bom yes) (on_board yes)
+    (property "Reference" "#PWR0110" (id 0) (at 181.356 30.48 0)
+      (effects (font (size 1.27 1.27)) hide)
+    )
+    (property "Value" "GND" (id 1) (at 180.34 30.48 90)
+      (effects (font (size 1.27 1.27)) (justify left))
+    )
+    (property "Footprint" "" (id 2) (at 187.706 30.48 0)
+      (effects (font (size 1.27 1.27)) hide)
+    )
+    (property "Datasheet" "" (id 3) (at 187.706 30.48 0)
+      (effects (font (size 1.27 1.27)) hide)
+    )
+    (pin "1")
   )
   (symbol (lib_id "power:GND") (at 170.688 108.712 90) (unit 1)
@@
       (effects (font (size 1.524 1.524)) (justify right))
     )
-    (property "Value" "LM74800QDRRRQ1" (id 1) (at 116.3574 55.9054 0)
+    (property "Value" "LM74800QDRRRQ1" (id 1) (at 116.586 53.086 0)
       (effects (font (size 1.524 1.524)) (justify right))
     )
@@
     (pin "12")
     (pin "13")
-    (pin "14")
-    (pin "15")
-    (pin "16")
     (pin "2")
     (pin "3")
@@
     (pin "2")
   )
-  (symbol (lib_id "power:GND") (at 187.706 30.48 270) (unit 1)
-    (in_bom yes) (on_board yes) (fields_autoplaced)
-    (property "Reference" "#PWR0110" (id 0) (at 181.356 30.48 0)
-      (effects (font (size 1.27 1.27)) hide)
-    )
-    (property "Value" "GND" (id 1) (at 184.5311 30.9138 90)
-      (effects (font (size 1.27 1.27)) (justify right))
-    )
-    (property "Footprint" "" (id 2) (at 187.706 30.48 0)
-      (effects (font (size 1.27 1.27)) hide)
-    )
-    (property "Datasheet" "" (id 3) (at 187.706 30.48 0)
-      (effects (font (size 1.27 1.27)) hide)
-    )
-    (pin "1")
-  )
   (sheet (at 183.2864 122.1232) (size 12.7 3.81) (fields_autoplaced)

Commit message: cleared all pcb drc errors and warnings
Connections:
- net GND: now also C19.2, C20.2, C21.2, C22.2, R32.2, R33.2, R34.2, U6.EPAD (SGND)
- net Vdd: now also Q5.5 (D), Q5.6 (D), Q5.7 (D), Q5.8 (D), Q5.9 (D), Q6.5 (D), Q6.6 (D), Q6.7 (D), Q6.8 (D), Q6.9 (D); no longer Q5.1 (S), Q5.2 (S), Q5.3 (S), Q6.1 (S), Q6.2 (S), Q6.3 (S)
- net Vin: now also Q6.1 (S), Q6.2 (S), Q6.3 (S); no longer Q6.5 (D), Q6.6 (D), Q6.7 (D), Q6.8 (D), Q6.9 (D)
- net at U8.13 (PAD): now also U8.14 (PAD), U8.15 (PAD), U8.16 (PAD)
- new net: Q5.1 (S), Q5.2 (S), Q5.3 (S), R13.1, TP4.1, U4.8 (IN+), U8.9 (OUT)
- no-connect marks 11 -> 10
Changed lines of the file:
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@@
     (title "Power Supply")
     (company "Buildbotics LLC")
-    (comment 1 "Copyrught (c) 2016-2022, Buildbotics LLC")
+    (comment 1 "Copyright (c) 2016-2022, Buildbotics LLC")
     (comment 2 "Licensed under CERN-OHL-S v2 ")
   )
@@
   (junction (at 272.542 140.716) (diameter 0) (color 0 0 0 0)
   )
+  (junction (at 126.238 161.036) (diameter 0) (color 0 0 0 0)
+  )
   (junction (at 110.744 36.322) (diameter 0) (color 0 0 0 0)
   )
@@
   (junction (at 43.7388 16.51) (diameter 0) (color 0 0 0 0)
   )
+  (junction (at 122.428 161.036) (diameter 0) (color 0 0 0 0)
+  )
   (junction (at 157.226 143.256) (diameter 0) (color 0 0 0 0)
   )
@@
   (junction (at 25.146 143.002) (diameter 0) (color 0 0 0 0)
   )
-  (no_connect (at 100.584 67.31))
   (no_connect (at 252.476 102.616))
   (no_connect (at 255.016 102.616))
@@
     (stroke (width 0) (type default) (color 0 0 0 0))
   )
-  (wire (pts (xy 100.584 65.532) (xy 100.584 67.31))
-    (stroke (width 0) (type default) (color 0 0 0 0))
-  )
   (wire (pts (xy 217.2716 117.856) (xy 217.2716 121.2088))
     (stroke (width 0) (type default) (color 0 0 0 0))
@@
     (stroke (width 0) (type default) (color 0 0 0 0))
   )
+  (wire (pts (xy 122.428 161.036) (xy 126.238 161.036))
+    (stroke (width 0) (type default) (color 0 0 0 0))
+  )
   (wire (pts (xy 34.544 143.002) (xy 25.146 143.002))
     (stroke (width 0) (type default) (color 0 0 0 0))
@@
     (pin "4")
   )
-  (symbol (lib_id "1LibBBCTRL:BSC040N08NS5ATMA1") (at 90.424 16.51 0) (mirror y) (unit 1)
+  (symbol (lib_name "BSC040N08NS5ATMA1_1") (lib_id "1LibBBCTRL:BSC040N08NS5ATMA1") (at 90.424 16.51 0) (mirror y) (unit 1)
     (in_bom yes) (on_board yes)
     (property "Reference" "Q6" (id 0) (at 85.0392 19.6596 0)
@@
     (pin "2")
   )
-  (symbol (lib_name "BSC040N08NS5ATMA1_1") (lib_id "1LibBBCTRL:BSC040N08NS5ATMA1") (at 120.904 16.51 0) (unit 1)
+  (symbol (lib_id "1LibBBCTRL:BSC040N08NS5ATMA1") (at 120.904 16.51 0) (unit 1)
     (in_bom yes) (on_board yes)
     (property "Reference" "Q5" (id 0) (at 127.254 20.1168 0)
@@
     (pin "12")
     (pin "13")
+    (pin "14")
+    (pin "15")
+    (pin "16")
     (pin "2")
     (pin "3")

Commit message: replaced some parts numbers with parts that are available
Parts:
- C12, C20, C21: value 1uF -> 1uF 100V
- C14: footprint Resistor_SMD:R_0805_2012Metric_Pad1.20x1.40mm_HandSolder -> Capacitor_SMD:C_0805_2012Metric_Pad1.18x1.45mm_HandSolder; Model CL21C131JBANNNC -> 08055A131JAT2A
- C19: value 10uF -> 10uF 63V
- C22: Model RC0805FR-07100KL -> CL21B223KBANNNC
- C23: Model C0805C104Z5VACTU -> C0805C104M5RACTU
- D1: Model (none) -> 5.0SMDJ48CA
- J2: Model (none) -> 39-30-0060
- Q5, Q6: Model (none) -> BSC040N08NS5ATMA1
- Q7, Q9: Model (none) -> 2N7002K
- Q8: Model (none) -> NTD5867NLT4G
- R14, R9: value 100k -> 100k .5%
- U2: Model (none) -> ATtiny1616-S
- Z1, Z2: Model (none) -> DDZ6V2BQ-7
Connections:
- net GND: now also C14.1; no longer C14.2
- net drv_enable_5V: now also C14.2; no longer C14.1

Commit message: corrections after first KiCad build
Parts:
- added R90: 1.82k, Resistor_SMD:R_0805_2012Metric_Pad1.20x1.40mm_HandSolder, symbol Device:R_US
- added TP15: Prog, Project_Footprints_Library:test_point, symbol Connector:TestPoint
- added TP24: Vin, Project_Footprints_Library:test_point, symbol Connector:TestPoint
- R35: value 422 -> 1.96k; Model RC0805FR-07422RL -> RC0805FR-071K96L
- TP1, TP10, TP11, TP13, TP14, TP3, TP4, TP6, TP8: footprint Connector_PinHeader_1.00mm:PinHeader_1x01_P1.00mm_Vertical -> Project_Footprints_Library:test_point
- TP5: value TP_Vs -> Vs; footprint Connector_PinHeader_1.00mm:PinHeader_1x01_P1.00mm_Vertical -> Project_Footprints_Library:test_point
Connections:
- net GND: now also R90.2
- net at R18.2, R19.1, U2.16 (~{RESET}/PA0): now also TP15.1
- net at C24.1, C25.1, C26.2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: now also R90.1
- net at C18.1, C19.1, C20.1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: now also TP24.1
- net 3to5_1/out renamed 3V_to_5V/out
- now unconnected: U8.13 (PAD)
- no-connect marks 10 -> 11
Other:
- removed sheet 3to5_1
- added sheet 3V_to_5V (level_shifter.kicad_sch)
- moved on the sheet: C11, C24, C26, R11, R12, R20, R35, TP3

Commit message: put all schematics on 50 mil grid
Other:
- moved on the sheet: C12, C13, C14, C97, D1, Q5, Q6, Q7, R10, R11, R12, R13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

Commit message: first commit of V18
Parts:
- added C87: .1uF, Capacitor_SMD:C_0805_2012Metric_Pad1.18x1.45mm_HandSolder, symbol Device:C
- added U10: SN74AHC1G125DBVR, Project_Footprints_Library:SN74AHC1G125DBVR, symbol 1LibBBCTRL:SN74AHC1G125DBVR
Connections:
- net +5V: now also C87.2, U10.5 (VCC)
- net GND: now also C87.1, U10.1 (*OE), U10.3 (GND)
- net pwr_tx: now also U10.2 (A)
- net 3V_to_5V/out: no longer names the net of R19.2
- net 3V_to_5V/out: now also U10.4 (Y)
Other:
- removed sheet 3V_to_5V
- moved on the sheet: J14

Commit message: added oled support
Changed lines of the file:
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@@
-    (stroke (width 0) (type default) (color 0 0 0 0))
-  )
-  (wire (pts (xy 191.77 146.05) (xy 192.024 145.796))
     (stroke (width 0) (type default) (color 0 0 0 0))
   )
@@
     (pin "2")
   )
-  (symbol (lib_id "power:GND") (at 192.024 145.796 0) (unit 1)
-    (in_bom yes) (on_board yes) (fields_autoplaced)
-    (property "Reference" "#PWR0127" (id 0) (at 192.024 152.146 0)
-      (effects (font (size 1.27 1.27)) hide)
-    )
-    (property "Value" "GND" (id 1) (at 192.024 150.2394 0))
-    (property "Footprint" "" (id 2) (at 192.024 145.796 0)
-      (effects (font (size 1.27 1.27)) hide)
-    )
-    (property "Datasheet" "" (id 3) (at 192.024 145.796 0)
-      (effects (font (size 1.27 1.27)) hide)
-    )
+  (symbol (lib_id "power:GND") (at 191.77 146.05 0) (unit 1)
+    (in_bom yes) (on_board yes) (fields_autoplaced)
+    (property "Reference" "#PWR0127" (id 0) (at 191.77 152.4 0)
+      (effects (font (size 1.27 1.27)) hide)
+    )
+    (property "Value" "GND" (id 1) (at 191.77 150.4934 0))
+    (property "Footprint" "" (id 2) (at 191.77 146.05 0)
+      (effects (font (size 1.27 1.27)) hide)
+    )
+    (property "Datasheet" "" (id 3) (at 191.77 146.05 0)
+      (effects (font (size 1.27 1.27)) hide)
+    )

Commit message: added some testpoints
Parts:
- TP2, TP7, TP9: footprint Connector_PinHeader_1.00mm:PinHeader_1x01_P1.00mm_Vertical -> Project_Footprints_Library:test_point
- U4: value TSC2012IDT -> TSC2012IYST; footprint Project_Footprints_Library:TSC2012IDT -> Package_SO:MSOP-8_3x3mm_P0.65mm; Model TSC2012IDT -> TSC2012IYST
- U8: value LM74800QDRRRQ1 -> LM74801QDRRRQ1; Model LM74800QDRRRQ1 -> LM74801QDRRRQ1
Changed lines of the file:
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@@
     (property "Reference" "TP2" (id 0) (at 113.538 28.702 90))
     (property "Value" "TP_HGATE" (id 1) (at 114.554 32.766 90))
-    (property "Footprint" "Connector_PinHeader_1.00mm:PinHeader_1x01_P1.00mm_Vertical" (id 2) (at 116.84 25.4 0)
+    (property "Footprint" "Project_Footprints_Library:test_point" (id 2) (at 116.84 25.4 0)
       (effects (font (size 1.27 1.27)) hide)
     )
@@
       (effects (font (size 1.524 1.524)))
     )
-    (property "Value" "LM74800QDRRRQ1" (id 1) (at 106.934 50.292 0)
+    (property "Value" "LM74801QDRRRQ1" (id 1) (at 106.934 50.292 0)
       (effects (font (size 1.524 1.524)))
     )
@@
       (effects (font (size 1.524 1.524)) hide)
     )
-    (property "Datasheet" "" (id 3) (at 100.838 57.15 0)
+    (property "Datasheet" "https://www.ti.com/lit/ds/symlink/lm7480-q1.pdf?HQS=dis-dk-null-digikeymode-dsf-pf-null-wwe&ts=1682672663618" (id 3) (at 100.838 57.15 0)
       (effects (font (size 1.524 1.524)) hide)
     )
-    (property "Model" "LM74800QDRRRQ1" (id 4) (at 83.82 8.89 0)
+    (property "Model" "LM74801QDRRRQ1" (id 4) (at 83.82 8.89 0)
       (effects (font (size 1.27 1.27)) hide)
     )
@@
       (effects (font (size 1.524 1.524)))
     )
-    (property "Value" "TSC2012IDT" (id 1) (at 209.804 27.432 0)
+    (property "Value" "TSC2012IYST" (id 1) (at 209.804 27.432 0)
       (effects (font (size 1.524 1.524)))
     )
-    (property "Footprint" "Project_Footprints_Library:TSC2012IDT" (id 2) (at 256.54 21.844 0)
+    (property "Footprint" "Package_SO:MSOP-8_3x3mm_P0.65mm" (id 2) (at 256.54 21.844 0)
       (effects (font (size 1.524 1.524)) hide)
     )
@@
       (effects (font (size 1.524 1.524)) hide)
     )
-    (property "Model" "TSC2012IDT" (id 4) (at 233.68 27.94 0)
+    (property "Model" "TSC2012IYST" (id 4) (at 233.68 27.94 0)
       (effects (font (size 1.27 1.27)) hide)
     )
@@
     (property "Reference" "TP9" (id 0) (at 71.374 149.86 0))
     (property "Value" "TP_FB" (id 1) (at 69.596 154.432 0))
-    (property "Footprint" "Connector_PinHeader_1.00mm:PinHeader_1x01_P1.00mm_Vertical" (id 2) (at 63.5 148.59 0)
+    (property "Footprint" "Project_Footprints_Library:test_point" (id 2) (at 63.5 148.59 0)
       (effects (font (size 1.27 1.27)) hide)
     )
@@
       (effects (font (size 1.27 1.27)) (justify left))
     )
-    (property "Footprint" "Connector_PinHeader_1.00mm:PinHeader_1x01_P1.00mm_Vertical" (id 2) (at 214.63 57.15 0)
-      (effects (font (size 1.27 1.27)) hide)
-    )
+    (property "Footprint" "Project_Footprints_Library:test_point" (id 2) (at 214.63 57.15 0)
+      (effects (font (size 1.27 1.27)) hide)
+    )
