File: PowerSupply.kicad_sch (KiCad schematic)
At the start: 89 parts, among them J14 PROG, J2 39-30-0060, J3 ENABLE, Q10 FDC5614P, Q5 BSC040N08NS5ATMA1, Q6 BSC040N08NS5ATMA1, Q7 2N7002K, Q8 NTD5867NLT4G, Q9 2N7002K, U10 SN74AHC1G125DBVR, U2 ATtiny1616-S, U4 TSC2012IYST, U6 L7987, U7 AZ1117IH-3.3TRG1, U8 LM74801QDRRRQ1

Commit message: corrected solder mask for Molex connectors
Parts:
- J2: footprint Molex-39-30-0060-* -> Project_Footprints_Library:Molex-39-30-0060-MFG
Changed lines of the file:
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@@
       (effects (font (size 1.27 1.27)) hide)
     )
-    (property "Footprint" "Molex-39-30-0060-*" (id 2) (at 39.37 27.94 0)
+    (property "Footprint" "Project_Footprints_Library:Molex-39-30-0060-MFG" (id 2) (at 39.37 27.94 0)
       (effects (font (size 1.27 1.27)) (justify left) hide)
     )
@@
       (effects (font (size 1.27 1.27)) (justify right) hide)
     )
-    (property "Footprint" "Molex-39-30-0060-*" (id 2) (at 19.05 27.94 0)
-      (effects (font (size 1.27 1.27)) (justify left) hide)
-    )
+    (property "Footprint" "Project_Footprints_Library:Molex-39-30-0060-MFG" (id 2) (at 19.05 27.94 0)
+      (effects (font (size 1.27 1.27)) (justify left) hide)
+    )

Commit message: updated some part numbers
Parts:
- R90: Model RC0805FR-071K82 -> RC0805FR-071K82L
Changed lines of the file:
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@@
       (effects (font (size 1.27 1.27)) hide)
     )
-    (property "Model" "RC0805FR-071K82" (id 4) (at 163.83 177.165 0)
+    (property "Model" "RC0805FR-071K82L" (id 4) (at 163.83 177.165 0)
       (effects (font (size 1.27 1.27)) hide)
     )

Commit message: Move back to drv8711
Parts:
- removed C87: .1uF, Capacitor_SMD:C_0805_2012Metric_Pad1.18x1.45mm_HandSolder, symbol Device:C
- removed D5: 12V, Package_TO_SOT_SMD:SOT-23, symbol Diode:BZX84Cxx
- removed U10: SN74AHC1G125DBVR, Project_Footprints_Library:SN74AHC1G125DBVR, symbol 1LibBBCTRL:SN74AHC1G125DBVR
- added Z4: 12V, Package_TO_SOT_SMD:SOT-23, symbol 1LibBBCTRL:MMBZ5242BLT3G
- C11: value ,68uF -> .68uF
- J2: footprint Project_Footprints_Library:Molex-39-30-0060-MFG -> Molex-39-30-0060-*
- R90: Model RC0805FR-071K82L -> RC0805FR-071K82
- TP2, TP7, TP9: footprint Project_Footprints_Library:test_point -> Connector_PinHeader_1.00mm:PinHeader_1x01_P1.00mm_Vertical
- U4: value TSC2012IYST -> TSC2012IDT; footprint Package_SO:MSOP-8_3x3mm_P0.65mm -> Project_Footprints_Library:TSC2012IDT; Model TSC2012IYST -> TSC2012IDT
Connections:
- net Vdd: now also Z4.3
- net 3V_to_5V/out: now reaches R19.2
- net at C17.1, Q10.3, R29.1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: now also Z4.1
Other:
- added sheet 3V_to_5V (level_shifter.kicad_sch)
- moved on the sheet: J14, L1

Commit message: All DRC errors cleared after conversion to Kicad V7
Parts:
- J2: footprint Molex-39-30-0060-* -> Project_Footprints_Library:Molex-39-30-0060-MFG
Other:
- moved on the sheet: C16, C17, C23, C27, C28, C29, D4, D6, J14, J3, Q9, R17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

Commit message: changed level shifter symbol
Parts:
- C22: Model CL21B223KBANNNC -> c0805c333k5ractu
Changed lines of the file:
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@@
       (effects (font (size 1.27 1.27)) hide)
     )
-    (property "Model" "CL21B223KBANNNC" (at 95.25 153.67 0)
+    (property "Model" "c0805c333k5ractu" (at 95.25 153.67 0)
       (effects (font (size 1.27 1.27)) hide)
     )
