File: PowerSupply.kicad_sch (KiCad schematic)
At the start: 87 parts, among them J14 PROG, J2 39-30-0060, J3 ENABLE, Q10 FDC5614P, Q5 BSC040N08NS5ATMA1, Q6 BSC040N08NS5ATMA1, Q7 2N7002K, Q8 NTD5867NLT4G, Q9 2N7002K, U2 ATtiny1616-S, U4 TSC2012IDT, U6 L7987, U7 AZ1117IH-3.3TRG1, U8 LM74801QDRRRQ1

Commit message: fixed footprint for q5 and q6, improved DRV8711 layout, oriented all 22uf caps the same direction
Parts:
- Q5, Q6: footprint INFINEON_PG-TDSON-8-5 -> Package_TO_SOT_SMD:TDSON-8-1
Changed lines of the file:
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@@
       (effects (font (size 1.27 1.27)) hide)
     )
-    (property "Footprint" "INFINEON_PG-TDSON-8-5" (at 142.24 13.97 0)
+    (property "Footprint" "Package_TO_SOT_SMD:TDSON-8-1" (at 142.24 13.97 0)
       (effects (font (size 1.27 1.27)) (justify left) hide)
     )
@@
       (effects (font (size 1.27 1.27)) hide)
     )
-    (property "Footprint" "INFINEON_PG-TDSON-8-5" (at 68.58 13.97 0)
-      (effects (font (size 1.27 1.27)) (justify left) hide)
-    )
+    (property "Footprint" "Package_TO_SOT_SMD:TDSON-8-1" (at 68.58 13.97 0)
+      (effects (font (size 1.27 1.27)) (justify left) hide)
+    )

Commit message: changed 12V supply for 0-10V out to LDO voltage regulator
Parts:
- Q5, Q6: footprint Package_TO_SOT_SMD:TDSON-8-1 -> INFINEON_PG-TDSON-8-5
Connections:
- net Vdd: no longer Q5.9 (D), Q6.9 (D)
Changed lines of the file:
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@@
       (effects (font (size 1.27 1.27)) hide)
     )
-    (property "Footprint" "Package_TO_SOT_SMD:TDSON-8-1" (at 142.24 13.97 0)
+    (property "Footprint" "INFINEON_PG-TDSON-8-5" (at 142.24 13.97 0)
       (effects (font (size 1.27 1.27)) (justify left) hide)
     )
@@
     (pin "7")
     (pin "8")
-    (pin "9")
     (instances
       (project "BuildboticsController"
@@
       (effects (font (size 1.27 1.27)) hide)
     )
-    (property "Footprint" "Package_TO_SOT_SMD:TDSON-8-1" (at 68.58 13.97 0)
+    (property "Footprint" "INFINEON_PG-TDSON-8-5" (at 68.58 13.97 0)
       (effects (font (size 1.27 1.27)) (justify left) hide)
     )
@@
     (pin "7")
     (pin "8")
-    (pin "9")
-    (instances
-      (project "BuildboticsController"
+    (instances
+      (project "BuildboticsController"

Commit message: make power_tx level shifter hard enabled
Parts:
- added C87: .1uF, Capacitor_SMD:C_0805_2012Metric_Pad1.18x1.45mm_HandSolder, symbol Device:C
- added U5: SN74AHC1G125DBVR, Project_Footprints_Library:SN74AHC1G125DBVR, symbol 1LibBBCTRL:SN74AHC1G125DBVR
Connections:
- net +5V: now also C87.2, U5.5 (VCC)
- net GND: now also C87.1, U5.1 (*OE), U5.3 (GND)
- net pwr_tx: now also U5.2 (A)
- net 3V_to_5V/out: no longer names the net of R19.2
- net 3V_to_5V/out: now also U5.4 (Y)
Other:
- removed sheet 3V_to_5V
- moved on the sheet: J14

Commit message: Replaced D6 with previous part and corrected R13 footprint
Parts:
- D6: value MBR0580 -> STPS3L60U; footprint Diode_SMD:D_SOD-123 -> Diode_SMD:D_2010_5025Metric; Model MBR0580S1-7 -> STPS3L60U
- R13: footprint Resistor_SMD:R_2512_6332Metric_Pad1.40x3.35mm_HandSolder -> Project_Footprints_Library:2512_Sense
- renumbered C87 to C92
Changed lines of the file:
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@@
   (symbol (lib_name "GND_1") (lib_id "power:GND") (at 187.96 110.49 0) (mirror x) (unit 1)
     (in_bom yes) (on_board yes) (dnp no) (fields_autoplaced)
-    (property "Reference" "#PWR0121" (at 187.96 104.14 0)
+    (property "Reference" "#PWR09" (at 187.96 104.14 0)
       (effects (font (size 1.27 1.27)) hide)
     )
@@
       (effects (font (size 1.27 1.27)) (justify left))
     )
-    (property "Value" "MBR0580" (at 159.512 149.9747 90)
-      (effects (font (size 1.27 1.27)) (justify left))
-    )
-    (property "Footprint" "Diode_SMD:D_SOD-123" (at 153.035 148.59 0)
-      (effects (font (size 1.27 1.27)) hide)
-    )
-    (property "Datasheet" "http://www.mccsemi.com/up_pdf/MBR0520~MBR0580(SOD123).pdf" (at 157.48 148.59 0)
-      (effects (font (size 1.27 1.27)) hide)
-    )
-    (property "Model" "MBR0580S1-7" (at 157.48 148.59 0)
+    (property "Value" "STPS3L60U" (at 159.512 149.9747 90)
+      (effects (font (size 1.27 1.27)) (justify left))
+    )
+    (property "Footprint" "Diode_SMD:D_2010_5025Metric" (at 153.035 148.59 0)
+      (effects (font (size 1.27 1.27)) hide)
+    )
+    (property "Datasheet" "https://www.mouser.com/datasheet/2/389/stps3l60-1851713.pdf" (at 157.48 148.59 0)
+      (effects (font (size 1.27 1.27)) hide)
+    )
+    (property "Model" "STPS3L60U" (at 157.48 148.59 0)
       (effects (font (size 1.27 1.27)) hide)
     )
@@
       (effects (font (size 1.27 1.27)))
     )
-    (property "Footprint" "Resistor_SMD:R_2512_6332Metric_Pad1.40x3.35mm_HandSolder" (at 204.47 17.78 90)
+    (property "Footprint" "Project_Footprints_Library:2512_Sense" (at 204.47 17.78 90)
       (effects (font (size 1.27 1.27)) hide)
     )
@@
   (symbol (lib_id "power:GND") (at 184.15 124.46 90) (unit 1)
     (in_bom yes) (on_board yes) (dnp no) (fields_autoplaced)
-    (property "Reference" "#PWR0122" (at 190.5 124.46 0)
+    (property "Reference" "#PWR08" (at 190.5 124.46 0)
       (effects (font (size 1.27 1.27)) hide)
     )
@@
   (symbol (lib_id "Device:C") (at 187.96 114.3 0) (unit 1)
     (in_bom yes) (on_board yes) (dnp no) (fields_autoplaced)
-    (property "Reference" "C87" (at 190.881 113.4653 0)
-      (effects (font (size 1.27 1.27)) (justify left))
-    )
+    (property "Reference" "C92" (at 190.881 113.4653 0)
+      (effects (font (size 1.27 1.27)) (justify left))
+    )
