File: MotorDriver.kicad_sch (KiCad schematic)
At the start: 26 parts, among them J1 43045-0402, Q1 NVMFD5C672NLT1G, Q2 NVMFD5C672NLT1G, Q3 NVMFD5C672NLT1G, Q4 NVMFD5C672NLT1G, U1 DRV8711DCP

Commit message: replaced some parts numbers with parts that are available
Parts:
- C7: value .22uF -> .22uF 100V
- C8: Model CL21B105KBFNNNE -> CC0805KKX7R7BB105
- C9: Model CL21B224KCFSNWE -> C0805C104M5RACTU
- J1: Model (none) -> 43045-0402
- Q1, Q2, Q3, Q4: Model (none) -> NVMFD5C672NLT1G
- R3, R5: Model CSR2512C0R05F -> CSRL3-0R05F8
Changed lines of the file:
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@@
       (effects (font (size 1.27 1.27)) hide)
     )
-    (property "Model" "CSR2512C0R05F" (id 4) (at 188.7728 149.86 0)
+    (property "Model" "CSRL3-0R05F8" (id 4) (at 188.7728 149.86 0)
       (effects (font (size 1.27 1.27)) hide)
     )
@@
   )
   (symbol (lib_id "Device:C") (at 98.552 151.13 0) (unit 1)
-    (in_bom yes) (on_board yes) (fields_autoplaced)
-    (property "Reference" "C7" (id 0) (at 101.473 150.2953 0)
-      (effects (font (size 1.27 1.27)) (justify left))
-    )
-    (property "Value" ".22uF" (id 1) (at 101.473 152.8322 0)
+    (in_bom yes) (on_board yes)
+    (property "Reference" "C7" (id 0) (at 91.948 148.844 0)
+      (effects (font (size 1.27 1.27)) (justify left))
+    )
+    (property "Value" ".22uF 100V" (id 1) (at 86.36 154.178 0)
       (effects (font (size 1.27 1.27)) (justify left))
     )
@@
       (effects (font (size 1.27 1.27)) (justify left) hide)
     )
+    (property "Model" "NVMFD5C672NLT1G" (id 46) (at 266.3444 63.4492 0)
+      (effects (font (size 1.27 1.27)) hide)
+    )
     (pin "1")
     (pin "2")
@@
       (effects (font (size 1.27 1.27)) (justify left) hide)
     )
+    (property "Model" "NVMFD5C672NLT1G" (id 46) (at 192.6844 63.4492 0)
+      (effects (font (size 1.27 1.27)) hide)
+    )
     (pin "1")
     (pin "2")
@@
       (effects (font (size 1.27 1.27)) (justify left) hide)
     )
+    (property "Model" "NVMFD5C672NLT1G" (id 46) (at 266.3444 63.4492 0)
+      (effects (font (size 1.27 1.27)) hide)
+    )
     (pin "1")
     (pin "2")
@@
       (effects (font (size 1.27 1.27)) (justify left) hide)
     )
+    (property "Model" "NVMFD5C672NLT1G" (id 46) (at 192.532 107.188 0)
+      (effects (font (size 1.27 1.27)) hide)
+    )
     (pin "1")
     (pin "2")
@@
       (effects (font (size 1.27 1.27)) (justify left) hide)
     )
+    (property "Model" "NVMFD5C672NLT1G" (id 46) (at 264.922 107.95 0)
+      (effects (font (size 1.27 1.27)) hide)
+    )
     (pin "1")
     (pin "2")
@@
     (property "voltage rating" "600V" (id 30) (at 143.1544 66.6242 0)
       (effects (font (size 1.27 1.27)) (justify left) hide)
+    )
+    (property "Model" "43045-0402" (id 31) (at 226.9744 66.6242 0)
+      (effects (font (size 0 0)) hide)
     )
     (pin "1")
@@
       (effects (font (size 1.27 1.27)) (justify left) hide)
     )
+    (property "Model" "43045-0402" (id 31) (at 226.9744 66.6242 0)
+      (effects (font (size 0 0)) hide)
+    )
     (pin "1")
     (pin "2")
@@
     (property "typ forward diode voltage" "0.9V" (id 45) (at 192.6844 -58.4708 0)
       (effects (font (size 1.27 1.27)) (justify left) hide)
+    )
+    (property "Model" "NVMFD5C672NLT1G" (id 46) (at 192.6844 63.4492 0)
+      (effects (font (size 1.27 1.27)) hide)
     )
     (pin "1")
@@
       (effects (font (size 1.27 1.27)) (justify left) hide)
     )
+    (property "Model" "NVMFD5C672NLT1G" (id 46) (at 192.532 107.188 0)
+      (effects (font (size 1.27 1.27)) hide)
+    )
     (pin "1")
     (pin "2")
@@
       (effects (font (size 1.27 1.27)) hide)
     )
-    (property "Model" "CSR2512C0R05F" (id 4) (at 181.864 101.6 0)
+    (property "Model" "CSRL3-0R05F8" (id 4) (at 181.864 101.6 0)
       (effects (font (size 1.27 1.27)) hide)
     )
@@
       (effects (font (size 1.27 1.27)) (justify left) hide)
     )
+    (property "Model" "NVMFD5C672NLT1G" (id 46) (at 264.922 107.95 0)
+      (effects (font (size 1.27 1.27)) hide)
+    )
     (pin "1")
     (pin "2")
@@
       (effects (font (size 1.27 1.27)) hide)
     )
-    (property "Model" "CL21B224KCFSNWE" (id 4) (at 106.172 71.12 0)
+    (property "Model" "C0805C104M5RACTU" (id 4) (at 106.172 71.12 0)
       (effects (font (size 1.27 1.27)) hide)
     )
@@
       (effects (font (size 1.27 1.27)) hide)
     )
-    (property "Model" "CL21B105KBFNNNE" (id 4) (at 104.648 162.56 0)
-      (effects (font (size 1.27 1.27)) hide)
-    )
+    (property "Model" "CC0805KKX7R7BB105" (id 4) (at 104.648 162.56 0)
+      (effects (font (size 1.27 1.27)) hide)
+    )

Commit message: corrections after first KiCad build
Parts:
- removed TP15: TP_STALL, Connector_PinHeader_1.00mm:PinHeader_1x01_P1.00mm_Vertical, symbol Connector:TestPoint
- removed TP16: TP_BEMF, Connector_PinHeader_1.00mm:PinHeader_1x01_P1.00mm_Vertical, symbol Connector:TestPoint
Changed lines of the file:
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@@
     (comment 2 "Licensed under CERN-OHL-S v2 ")
   )
-  (junction (at 170.942 154.94) (diameter 0) (color 0 0 0 0)
-  )
   (junction (at 170.5356 101.6) (diameter 0) (color 0 0 0 0)
   )
@@
   )
   (junction (at 181.102 149.86) (diameter 0) (color 0 0 0 0)
-  )
-  (junction (at 98.5012 137.16) (diameter 0) (color 0 0 0 0)
   )
   (junction (at 254.254 21.6408) (diameter 0) (color 0 0 0 0)
@@
   (no_connect (at 109.982 101.6))
   (no_connect (at 109.982 104.14))
-  (wire (pts (xy 98.5012 137.16) (xy 109.982 137.16))
+  (wire (pts (xy 94.996 137.16) (xy 109.982 137.16))
     (stroke (width 0) (type default) (color 0 0 0 0))
   )
@@
   )
   (wire (pts (xy 267.0048 30.0736) (xy 267.0048 29.21))
-    (stroke (width 0) (type default) (color 0 0 0 0))
-  )
-  (wire (pts (xy 94.996 137.16) (xy 98.5012 137.16))
     (stroke (width 0) (type default) (color 0 0 0 0))
   )
@@
     (pin "2")
   )
-  (symbol (lib_id "Connector:TestPoint") (at 170.942 154.94 270) (unit 1)
-    (in_bom yes) (on_board yes) (fields_autoplaced)
-    (property "Reference" "TP16" (id 0) (at 175.641 154.1053 90)
-      (effects (font (size 1.27 1.27)) (justify left))
-    )
-    (property "Value" "TP_BEMF" (id 1) (at 175.641 156.6422 90)
-      (effects (font (size 1.27 1.27)) (justify left))
-    )
-    (property "Footprint" "Connector_PinHeader_1.00mm:PinHeader_1x01_P1.00mm_Vertical" (id 2) (at 170.942 160.02 0)
-      (effects (font (size 1.27 1.27)) hide)
-    )
-    (property "Datasheet" "~" (id 3) (at 170.942 160.02 0)
-      (effects (font (size 1.27 1.27)) hide)
-    )
-    (pin "1")
-  )
   (symbol (lib_id "Device:C_Polarized_US") (at 267.0556 25.4 0) (unit 1)
     (in_bom yes) (on_board yes) (fields_autoplaced)
@@
     (pin "5-6")
   )
-  (symbol (lib_id "Connector:TestPoint") (at 98.5012 137.16 0) (unit 1)
-    (in_bom yes) (on_board yes) (fields_autoplaced)
-    (property "Reference" "TP15" (id 0) (at 99.8982 133.0233 0)
-      (effects (font (size 1.27 1.27)) (justify left))
-    )
-    (property "Value" "TP_STALL" (id 1) (at 99.8982 135.5602 0)
-      (effects (font (size 1.27 1.27)) (justify left))
-    )
-    (property "Footprint" "Connector_PinHeader_1.00mm:PinHeader_1x01_P1.00mm_Vertical" (id 2) (at 103.5812 137.16 0)
-      (effects (font (size 1.27 1.27)) hide)
-    )
-    (property "Datasheet" "~" (id 3) (at 103.5812 137.16 0)
-      (effects (font (size 1.27 1.27)) hide)
-    )
-    (pin "1")
-  )
   (symbol (lib_id "Device:C") (at 106.172 59.69 0) (unit 1)

Commit message: put all schematics on 50 mil grid
Other:
- moved on the sheet: C8, J1A, Q3A, Q4A

Commit message: first commit of V18
Parts:
- removed C10: 1uF, Capacitor_SMD:C_0805_2012Metric_Pad1.18x1.45mm_HandSolder, symbol Device:C
- removed C4, C5: 22uF, Capacitor_THT:CP_Radial_D5.0mm_P2.00mm, symbol Device:C_Polarized_US
- removed Q1, Q2, Q3, Q4: NVMFD5C672NLT1G, Project_Footprints_Library:ON_Semiconductor-506BT-02_2013-E-MFG, symbol 1LibBBCTRL:NVMFD5C672NLT1G
- removed R4, R6: 75, Resistor_SMD:R_0805_2012Metric_Pad1.20x1.40mm_HandSolder, symbol Device:R_US
- removed R5: .05, Resistor_SMD:R_2512_6332Metric_Pad1.40x3.35mm_HandSolder, symbol Device:R_US
- removed R7: 2.4k, Resistor_SMD:R_0805_2012Metric_Pad1.20x1.40mm_HandSolder, symbol Device:R_US
- removed R8: 180, Resistor_SMD:R_0805_2012Metric_Pad1.20x1.40mm_HandSolder, symbol Device:R_US
- removed U1: DRV8711DCP, Project_Footprints_Library:DRV8711DCP, symbol 1LibBBCTRL:DRV8711DCP
- added C38, C39: .01u, Capacitor_SMD:C_0805_2012Metric_Pad1.18x1.45mm_HandSolder, symbol Device:C
- added TP12: TP_nHOME, Project_Footprints_Library:test_point, symbol Connector:TestPoint
- added TP16: TP_nFAULT, Project_Footprints_Library:test_point, symbol Connector:TestPoint
- added U28: DRV8462DDWR, Project_Footprints_Library:DDW44_8P26X4P31, symbol 1LibBBCTRL:DRV8462DDWR
- C1: value 1nF -> C; Model C0805C102K4RACTU -> CL21B104KCFNNNE
- C6: value 10n -> .1u; Model C0805C103K1RAC7210 -> 08056D104KAT2A
- C7: value .22uF 100V -> 1u; Model CL21B224KCFSNWE -> CC0805KKX5R5BB105
- C8: value 1uF -> 1u; Model CC0805KKX7R7BB105 -> CL05A104KA5NNNC
- C9: value .1uF -> .01u; Model C0805C104M5RACTU -> CAP CER 10000PF 100V X7R 0805
- R1, R2: value 75 -> 10k; Model RMCF0805JT75R0 -> RC0805FR-0710KL
- R3: value .05 -> 10k; footprint Resistor_SMD:R_2512_6332Metric_Pad1.40x3.35mm_HandSolder -> Resistor_SMD:R_0805_2012Metric_Pad1.20x1.40mm_HandSolder; Model CSRL3-0R05F8 -> RC0805FR-0710KL
Connections:
- net +3.3V: now also R1.1, R2.1, R3.1
- net GND: now also C7.1, C9.2, C38.2, C39.1, U28.10 (PGNDA), U28.13 (PGNDB), U28.20 (PGNDB), U28.22 (GND), U28.23 (GND), U28.3 (PGNDA), U28.EPAD; no longer C1.2, C9.1, R3.1
- net Vs: now also C8.1, C9.1, C38.1, C39.2, U28.11 (VM), U28.12 (VM), U28.2 (VM), U28.21 (VM); no longer C6.2, C8.2
- net cs: now also U28.34 (nSCS/M0)
- net dir: now also U28.40 (DIR)
- net enable: now also U28.41 (ENABLE)
- net miso: now also U28.36 (SDO/DECAY1)
- net mosi: now also U28.37 (SDI/DECAY0)
- net sck: now also U28.38 (SCLK/M1)
- net step: now also U28.39 (STEP)
- net at C7.2: now also U28.24 (DVDD)
- net at C1.1: now also U28.44 (CPH)
- net at J1.2: now also U28.14 (BOUT2), U28.15 (BOUT2), U28.16 (BOUT2)
- net at R2.2: now also TP12.1, U28.27 (nHOME)
- net nFAULT: now reaches R3.2
- net nFAULT: now also TP16.1, U28.26 (nFAULT)
- net at J1.1: now also U28.17 (BOUT1), U28.18 (BOUT1), U28.19 (BOUT1)
- net at R1.2: now also U28.28 (MODE)
- net at J1.3: now also U28.7 (AOUT2), U28.8 (AOUT2), U28.9 (AOUT2)
- net at J1.4: now also U28.4 (AOUT1), U28.5 (AOUT1), U28.6 (AOUT1)
- new net: C6.2, U28.25 (VCC)
- new net: C8.2, U28.1 (VCP)
- new net: C1.2, U28.43 (CPL)
- new net nSLEEP: U28.42 (nSLEEP)
- no-connect marks 3 -> 6
Other:
- moved on the sheet: C2, C3, J1B

Commit message: motor driver improvements including corrected cap P/N, connected 3.3V to Vcc, and added exposed copper plane on back
Parts:
- C1: value C -> .1uF
- C8: Model CL05A104KA5NNNC -> CL21B105KOFNNNE
Connections:
- net +3.3V: now also C6.2, U28.25 (VCC)
Other:
- moved on the sheet: C6, R1, R2, R3, TP12, TP16

Commit message: updated some part numbers
Parts:
- C38, C39, C9: Model CAP CER 10000PF 100V X7R 0805 -> CL21B103KCANNNC
Changed lines of the file:
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@@
       (effects (font (size 1.27 1.27)) hide)
     )
-    (property "Model" "CAP CER 10000PF 100V X7R 0805" (id 4) (at 167.005 87.63 0)
+    (property "Description" "CAP CER 10000PF 100V X7R 0805" (id 4) (at 167.005 87.63 0)
+      (effects (font (size 1.27 1.27)) hide)
+    )
+    (property "Model" "CL21B103KCANNNC" (id 5) (at 167.005 87.63 90)
       (effects (font (size 1.27 1.27)) hide)
     )
@@
       (effects (font (size 1.27 1.27)) hide)
     )
-    (property "Model" "CAP CER 10000PF 100V X7R 0805" (id 4) (at 167.64 109.22 0)
+    (property "Description" "CAP CER 10000PF 100V X7R 0805" (id 4) (at 167.64 109.22 0)
+      (effects (font (size 1.27 1.27)) hide)
+    )
+    (property "Model" "CL21B103KCANNNC" (id 5) (at 167.64 109.22 90)
       (effects (font (size 1.27 1.27)) hide)
     )
@@
       (effects (font (size 1.27 1.27)) hide)
     )
-    (property "Model" "CAP CER 10000PF 100V X7R 0805" (id 4) (at 166.37 63.5 0)
-      (effects (font (size 1.27 1.27)) hide)
-    )
+    (property "Description" "CAP CER 10000PF 100V X7R 0805" (id 4) (at 166.37 63.5 0)
+      (effects (font (size 1.27 1.27)) hide)
+    )
+    (property "Model" "CL21B103KCANNNC" (id 5) (at 166.37 63.5 90)
+      (effects (font (size 1.27 1.27)) hide)
+    )

Commit message: Move back to drv8711
Parts:
- removed C38, C39: .01u, Capacitor_SMD:C_0805_2012Metric_Pad1.18x1.45mm_HandSolder, symbol Device:C
- removed TP12: TP_nHOME, Project_Footprints_Library:test_point, symbol Connector:TestPoint
- removed TP16: TP_nFAULT, Project_Footprints_Library:test_point, symbol Connector:TestPoint
- removed U28: DRV8462DDWR, Project_Footprints_Library:DDW44_8P26X4P31, symbol 1LibBBCTRL:DRV8462DDWR
- added C10: 1uF, Capacitor_SMD:C_0805_2012Metric_Pad1.18x1.45mm_HandSolder, symbol Device:C
- added C4, C5: 22uF, Capacitor_THT:CP_Radial_D5.0mm_P2.00mm, symbol Device:C_Polarized_US
- added Q1, Q2, Q3, Q4: DMTH6010LPD-13, Project_Footprints_Library:ON_Semiconductor-506BT-02_2013-E-MFG, symbol 1LibBBCTRL:NVMFD5C672NLT1G
- added R4, R6: 75, Resistor_SMD:R_0805_2012Metric_Pad1.20x1.40mm_HandSolder, symbol Device:R_US
- added R5: .05, Resistor_SMD:R_2512_6332Metric_Pad1.40x3.35mm_HandSolder, symbol Device:R_US
- added R7: 2.4k, Resistor_SMD:R_0805_2012Metric_Pad1.20x1.40mm_HandSolder, symbol Device:R_US
- added R8: 180, Resistor_SMD:R_0805_2012Metric_Pad1.20x1.40mm_HandSolder, symbol Device:R_US
- added U1: DRV8711DCP, Project_Footprints_Library:DRV8711DCP, symbol 1LibBBCTRL:DRV8711DCP
- C1: value .1uF -> 1nF; Model CL21B104KCFNNNE -> C0805C102K4RACTU
- C6: value .1u -> 10n; Model 08056D104KAT2A -> C0805C103K1RAC7210
- C7: value 1u -> .22uF 100V; Model CC0805KKX5R5BB105 -> CL21B224KCFSNWE
- C8: value 1u -> 1uF; Model CL21B105KOFNNNE -> CC0805KKX7R7BB105
- C9: value .01u -> .1uF; Model CL21B103KCANNNC -> C0805C104M5RACTU
- R1, R2: value 10k -> 75; Model RC0805FR-0710KL -> RMCF0805JT75R0
- R3: value 10k -> .05; footprint Resistor_SMD:R_0805_2012Metric_Pad1.20x1.40mm_HandSolder -> Resistor_SMD:R_2512_6332Metric_Pad1.40x3.35mm_HandSolder; Model RC0805FR-0710KL -> CSRL3-0R05F8
Connections:
- net +3.3V: now also R7.1; no longer C6.2, R1.1, R2.1, R3.1
- net GND: now also C1.2, C9.1, R3.1, C10.1, C4.2, C5.2, R5.1, U1.24 (BISENN), U1.29 (GND), U1.33 (AISENN), U1.38 (GND), U1.39 (PAD), U1.5 (GND); no longer C7.1, C9.2
- net Vs: now also C6.2, C8.2, C4.1, C5.1, Q1.7-8 (D1), Q2.5-6 (D2), Q3.7-8 (D1), Q4.5-6 (D2), U1.4 (VM); no longer C8.1, C9.1
- net cs: now also U1.16 (SCS)
- net dir: now also U1.11 (DIR_AIN2)
- net enable: now also U1.8 (SLEEP_N)
- net miso: now also U1.17 (SDATO)
- net mosi: now also U1.15 (SDATI)
- net sck: now also U1.14 (SCLK)
- net step: now also U1.10 (STEP_AIN1)
- net at R2.2: now also Q1.4 (G2)
- net at J1.1: now also Q1.1 (S1), Q1.5-6 (D2), U1.37 (AOUT1)
- net at J1.2: now also Q2.3 (S2), Q2.7-8 (D1), U1.30 (AOUT2)
- net at C7.2: now also U1.2 (CP2)
- net at C1.1: now also U1.20 (BEMF)
- net at J1.3: now also Q3.1 (S1), Q3.5-6 (D2), U1.28 (BOUT1)
- net at J1.4: now also Q4.3 (S2), Q4.7-8 (D1), U1.21 (BOUT2)
- net at R1.2: now also Q2.2 (G1)
- net nFAULT: no longer names the net of R3.2
- net nFAULT: now also Q1.3 (S2), Q2.1 (S1), U1.34 (AISENP)
- new net: Q3.3 (S2), Q4.1 (S1), R5.2, U1.25 (BISENP)
- new net: R6.1, U1.23 (B2LS)
- new net: Q4.2 (G1), R6.2
- new net: C7.1, U1.1 (CP1)
- new net: C10.2, U1.7 (VINT)
- new net: R7.2, R8.2, U1.19 (STALL_BEMFV_N)
- new net: R2.1, U1.35 (A1LS)
- new net: Q3.2 (G1), U1.27 (B1HS)
- new net: Q3.4 (G2), R4.2
- new net: Q2.4 (G2), U1.31 (A2HS)
- new net: Q4.4 (G2), U1.22 (B2HS)
- new net: R4.1, U1.26 (B1LS)
- new net: C8.1, U1.3 (VCP)
- new net: R1.1, U1.32 (A2LS)
- new net: Q1.2 (G1), U1.36 (A1HS)
- new net: C9.2, U1.6 (V5)
- new net fault: U1.18 (FAULT_N)
- new net stall: R8.1
- no-connect marks 6 -> 3
Other:
- moved on the sheet: C2, C3, J1B
