File: MotorDriver.kicad_sch (KiCad schematic)
At the start: 24 parts, among them J1 43045-0402, Q1 DMTH6010LPD-13, Q2 DMTH6010LPD-13, Q3 DMTH6010LPD-13, Q4 DMTH6010LPD-13, U1 DRV8711DCP

Commit message: All DRC errors cleared after conversion to Kicad V7
Connections:
- net GND: no longer C1.2, U1.29 (GND)
- new net: C1.2, U1.29 (GND)
Other:
- moved on the sheet: C1, C10, C3, C4, C5, C6, C7, C9, J1A, J1B, Q1A, Q1B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

Commit message: changed level shifter symbol
Connections:
- net GND: now also C1.2, U1.29 (GND)
Changed lines of the file:
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@@
   (junction (at 168.91 165.1) (diameter 0) (color 0 0 0 0)
+  )
+  (junction (at 168.91 162.56) (diameter 0) (color 0 0 0 0)
   )
   (junction (at 229.87 58.42) (diameter 0) (color 0 0 0 0)
@@
     (stroke (width 0) (type default))
   )
+  (wire (pts (xy 168.91 162.56) (xy 173.99 162.56))
+    (stroke (width 0) (type default))
+  )
   (wire (pts (xy 262.89 119.38) (xy 262.89 137.16))
     (stroke (width 0) (type default))
@@
     (stroke (width 0) (type default))
   )
-  (wire (pts (xy 168.91 160.02) (xy 168.91 165.1))
+  (wire (pts (xy 168.91 160.02) (xy 168.91 162.56))
     (stroke (width 0) (type default))
   )
@@
     (stroke (width 0) (type default))
   )
-  (wire (pts (xy 166.37 162.56) (xy 173.99 162.56))
-    (stroke (width 0) (type default))
-  )
   (wire (pts (xy 166.37 160.02) (xy 168.91 160.02))
     (stroke (width 0) (type default))
@@
     (stroke (width 0) (type default))
   )
+  (wire (pts (xy 166.37 162.56) (xy 168.91 162.56))
+    (stroke (width 0) (type default))
+  )
   (wire (pts (xy 185.42 119.38) (xy 194.31 119.38))
     (stroke (width 0) (type default))
@@
     (stroke (width 0) (type default))
   )
+  (wire (pts (xy 168.91 162.56) (xy 168.91 165.1))
+    (stroke (width 0) (type default))
+  )

Commit message: adjusted footprint and position motor port connectors
Parts:
- J1: footprint Project_Footprints_Library:Molex-43045-0402-MFG -> Project_Footprints_Library:CON_430450402_MOL
Changed lines of the file:
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@@
       (effects (font (size 1.27 1.27)) hide)
     )
-    (property "Footprint" "Project_Footprints_Library:Molex-43045-0402-MFG" (at 214.63 66.04 0)
+    (property "Footprint" "Project_Footprints_Library:CON_430450402_MOL" (at 214.63 66.04 0)
       (effects (font (size 1.27 1.27)) (justify left) hide)
     )
@@
       (effects (font (size 1.27 1.27)) (justify right) hide)
     )
-    (property "Footprint" "Project_Footprints_Library:Molex-43045-0402-MFG" (at 214.63 113.03 0)
-      (effects (font (size 1.27 1.27)) (justify left) hide)
-    )
+    (property "Footprint" "Project_Footprints_Library:CON_430450402_MOL" (at 214.63 113.03 0)
+      (effects (font (size 1.27 1.27)) (justify left) hide)
+    )
