File: rpi.kicad_sch (KiCad schematic)
At the start: 10 parts, among them J10 RPI, J11 SERIAL, J12 I2C, J13 LCD, Q23 2N7002K, Q24 2N7002K

Commit message: replaced some parts numbers with parts that are available
Parts:
- Q23, Q24: Model (none) -> 2N7002K
Changed lines of the file:
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@@
       (effects (font (size 1.27 1.27)) (justify left) hide)
+    )
+    (property "Model" "2N7002K" (id 4) (at 148.336 121.92 0)
+      (effects (font (size 1.27 1.27)) hide)
     )
     (pin "1")
@@
       (effects (font (size 1.27 1.27)) (justify left) hide)
     )
-    (pin "1")
+    (property "Model" "2N7002K" (id 4) (at 148.082 96.266 0)
+      (effects (font (size 1.27 1.27)) hide)
+    )
+    (pin "1")

Commit message: corrections after first KiCad build
Changed lines of the file:
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@@
     (stroke (width 0) (type default) (color 0 0 0 0))
-  )
-  (label "5V_scl" (at 197.612 111.252 0)
-    (effects (font (size 1.27 1.27)) (justify left bottom))
-  )
-  (label "5V_sda" (at 197.104 108.712 0)
-    (effects (font (size 1.27 1.27)) (justify left bottom))
   )
   (global_label "+5V" (shape input) (at 163.576 90.424 90) (fields_autoplaced)
@@
     (effects (font (size 1.27 1.27)) (justify right))
   )
+  (hierarchical_label "5V_sda" (shape output) (at 190.5 99.06 0)
+    (effects (font (size 1.27 1.27)) (justify left))
+  )
   (hierarchical_label "sda" (shape bidirectional) (at 118.364 96.774 90)
     (effects (font (size 1.27 1.27)) (justify left))
@@
     (effects (font (size 1.27 1.27)) (justify right))
   )
+  (hierarchical_label "5V_scl" (shape output) (at 190.754 124.206 0)
+    (effects (font (size 1.27 1.27)) (justify left))
+  )
   (hierarchical_label "serial_rx" (shape input) (at 90.678 101.092 0)

Commit message: put all schematics on 50 mil grid
Other:
- moved on the sheet: J10, J11

Commit message: minor corrections in prep for new build
Parts:
- J11, J12: Model Do Not Populate -> 68001-403HLF
Changed lines of the file:
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@@
       (effects (font (size 1.27 1.27)) hide)
     )
-    (property "Model" "Do Not Populate" (id 4) (at 96.52 116.84 0)
+    (property "Model" "68001-403HLF" (id 4) (at 96.52 116.84 0)
       (effects (font (size 1.27 1.27)) hide)
     )
@@
       (effects (font (size 1.27 1.27)) hide)
     )
-    (property "Model" "Do Not Populate" (id 4) (at 104.902 105.664 0)
+    (property "Model" "68001-403HLF" (id 4) (at 104.902 105.664 0)
       (effects (font (size 1.27 1.27)) hide)
     )

Commit message: added resistor to pull gpio 17 low to show board type
Parts:
- added R45: 1k, Resistor_SMD:R_0805_2012Metric_Pad1.20x1.40mm_HandSolder, symbol Device:R_US
Connections:
- net GND: now also R45.1
- net at J10.11 (Pin_11): now also R45.2
- no-connect marks 22 -> 21
Other:
- note added: "Note GPIO 17, 22, and 26 (pins 11,15, and 37 respectively) are pulled low in various combinations to signal the type of board. Pin 11 = L, Pin 15 = X, and Pin 37 = X) means that this board uses the new DRV8642 drivers."
Changed lines of the file:
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@@
   (no_connect (at 64.77 116.84))
   (no_connect (at 64.77 91.44))
-  (no_connect (at 64.77 104.14))
+  (no_connect (at 77.47 116.84))
   (no_connect (at 77.47 121.92))
   (no_connect (at 77.47 119.38))
@@
   (no_connect (at 77.47 124.46))
   (no_connect (at 77.47 111.76))
-  (no_connect (at 77.47 116.84))
   (no_connect (at 64.77 137.16))
   (no_connect (at 64.77 134.62))
@@
     (stroke (width 0) (type default) (color 0 0 0 0))
   )
+  (wire (pts (xy 57.785 104.14) (xy 64.77 104.14))
+    (stroke (width 0) (type default) (color 0 0 0 0))
+  )
   (wire (pts (xy 115.316 103.124) (xy 109.982 103.124))
     (stroke (width 0) (type default) (color 0 0 0 0))
@@
   (wire (pts (xy 131.318 109.982) (xy 131.318 112.776))
     (stroke (width 0) (type default) (color 0 0 0 0))
+  )
+  (text "Note GPIO 17, 22, and 26  (pins 11,15, and 37\nrespectively) are pulled low in various\ncombinations to signal the type of board.\nPin 11 = L, Pin 15 = X, and Pin 37 = X) means\nthat this board uses the new DRV8642 drivers."
+    (at 19.685 118.745 0)
+    (effects (font (size 1 1)) (justify left bottom))
   )
   (global_label "+5V" (shape input) (at 163.576 90.424 90) (fields_autoplaced)
@@
     (pin "3")
   )
+  (symbol (lib_id "Device:R_US") (at 53.975 104.14 90) (unit 1)
+    (in_bom yes) (on_board yes)
+    (property "Reference" "R45" (id 0) (at 48.895 100.965 90)
+      (effects (font (size 1.27 1.27)) (justify right))
+    )
+    (property "Value" "1k" (id 1) (at 52.2728 105.791 0)
+      (effects (font (size 1.27 1.27)) (justify right))
+    )
+    (property "Footprint" "Resistor_SMD:R_0805_2012Metric_Pad1.20x1.40mm_HandSolder" (id 2) (at 54.229 103.124 90)
+      (effects (font (size 1.27 1.27)) hide)
+    )
+    (property "Datasheet" "~" (id 3) (at 53.975 104.14 0)
+      (effects (font (size 1.27 1.27)) hide)
+    )
+    (property "Model" "RC0805FR-071KL" (id 4) (at 53.975 104.14 0)
+      (effects (font (size 1.27 1.27)) hide)
+    )
+    (pin "1")
+    (pin "2")
+  )
   (symbol (lib_id "Device:R_US") (at 163.83 119.888 0) (unit 1)
     (in_bom yes) (on_board yes) (fields_autoplaced)
@@
     )
     (property "Datasheet" "" (id 3) (at 64.77 101.6 0)
+      (effects (font (size 1.27 1.27)) hide)
+    )
+    (pin "1")
+  )
+  (symbol (lib_id "power:GND") (at 50.165 104.14 270) (unit 1)
+    (in_bom yes) (on_board yes)
+    (property "Reference" "#PWR0103" (id 0) (at 43.815 104.14 0)
+      (effects (font (size 1.27 1.27)) hide)
+    )
+    (property "Value" "GND" (id 1) (at 50.165 106.68 0))
+    (property "Footprint" "" (id 2) (at 50.165 104.14 0)
+      (effects (font (size 1.27 1.27)) hide)
+    )
+    (property "Datasheet" "" (id 3) (at 50.165 104.14 0)
       (effects (font (size 1.27 1.27)) hide)
     )
@@
   )
   (symbol (lib_id "power:GND") (at 77.47 127 90) (unit 1)
-    (in_bom yes) (on_board yes) (fields_autoplaced)
+    (in_bom yes) (on_board yes)
     (property "Reference" "#PWR0221" (id 0) (at 83.82 127 0)
       (effects (font (size 1.27 1.27)) hide)
     )
-    (property "Value" "GND" (id 1) (at 80.645 127.4338 90)
-      (effects (font (size 1.27 1.27)) (justify right))
-    )
+    (property "Value" "GND" (id 1) (at 80.645 128.27 90)
+      (effects (font (size 1.27 1.27)) (justify right))
+    )

Commit message: added oled support
Parts:
- added J16: OLED, Connector_PinHeader_2.54mm:PinHeader_1x04_P2.54mm_Vertical, symbol Connector_Generic:Conn_01x04
Connections:
- net +3.3V: now also J16.2 (Pin_2)
- net GND: now also J16.1 (Pin_1)
- net scl: now also J16.3 (Pin_3)
- net sda: now also J16.4 (Pin_4)
Other:
- moved on the sheet: J12, J13, Q23, Q24, R84, R85, R86, R87

Commit message: Move back to drv8711
Parts:
- removed J16: OLED, Connector_PinHeader_2.54mm:PinHeader_1x04_P2.54mm_Vertical, symbol Connector_Generic:Conn_01x04
- removed R45: 1k, Resistor_SMD:R_0805_2012Metric_Pad1.20x1.40mm_HandSolder, symbol Device:R_US
Connections:
- no-connect marks 21 -> 22
Other:
- note removed: "Note GPIO 17, 22, and 26 (pins 11,15, and 37 respectively) are pulled low in various combinations to signal the type of board. Pin 11 = L, Pin 15 = X, and Pin 37 = X) means that this board uses the new DRV8642 drivers."
- moved on the sheet: J12, J13, Q23, Q24, R84, R85, R86, R87
