File: rpi.kicad_sch (KiCad schematic)
At the start: 10 parts, among them J10 RPI, J11 SERIAL, J12 I2C, J13 LCD, Q23 2N7002K, Q24 2N7002K

Commit message: All DRC errors cleared after conversion to Kicad V7
Other:
- moved on the sheet: J12, J13, Q23, Q24, R85, R86, R87
