File: level_shifter.kicad_sch (KiCad schematic)
At the start: 2 parts, among them U5 SN74AHC1G125DBVR

Commit message: replaced some parts numbers with parts that are available
Parts:
- C15: value ~ -> .1uF
Changed lines of the file:
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@@
       (effects (font (size 1.27 1.27)) (justify left))
     )
-    (property "Value" "~" (id 1) (at 172.847 76.8862 0)
+    (property "Value" ".1uF" (id 1) (at 172.847 76.8862 0)
       (effects (font (size 1.27 1.27)) (justify left))
     )

Commit message: modified file to allow floating 5V buffer oe inputs until boot completes.
Connections:
- net GND: no longer U5.1 (*OE)
- new net buffer_enable: U5.1 (*OE)
Changed lines of the file:
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@@
     (stroke (width 0) (type default) (color 0 0 0 0))
+  )
+  (wire (pts (xy 106.68 83.566) (xy 109.728 83.566))
+    (stroke (width 0) (type default) (color 0 0 0 0))
+  )
+  (global_label "buffer_enable" (shape input) (at 106.68 83.566 180) (fields_autoplaced)
+    (effects (font (size 1.27 1.27)) (justify right))
+    (property "Intersheet References" "${INTERSHEET_REFS}" (id 0) (at 91.3855 83.4866 0)
+      (effects (font (size 1.27 1.27)) (justify right) hide)
+    )
   )
   (global_label "+5V" (shape input) (at 188.214 83.566 0) (fields_autoplaced)
@@
     (effects (font (size 1.27 1.27)) (justify left))
   )
-  (symbol (lib_id "power:GND") (at 109.728 83.566 270) (unit 1)
-    (in_bom yes) (on_board yes) (fields_autoplaced)
-    (property "Reference" "#PWR0122" (id 0) (at 103.378 83.566 0)
-      (effects (font (size 1.27 1.27)) hide)
-    )
-    (property "Value" "GND" (id 1) (at 106.5531 83.9998 90)
-      (effects (font (size 1.27 1.27)) (justify right))
-    )
-    (property "Footprint" "" (id 2) (at 109.728 83.566 0)
-      (effects (font (size 1.27 1.27)) hide)
-    )
-    (property "Datasheet" "" (id 3) (at 109.728 83.566 0)
-      (effects (font (size 1.27 1.27)) hide)
-    )
-    (pin "1")
-  )
   (symbol (lib_id "1LibBBCTRL:SN74AHC1G125DBVR") (at 109.728 83.566 0) (unit 1)

Commit message: corrections after first KiCad build
Parts:
- renumbered C15 to C87, U5 to U10
Changed lines of the file:
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@@
   (symbol (lib_id "1LibBBCTRL:SN74AHC1G125DBVR") (at 109.728 83.566 0) (unit 1)
     (in_bom yes) (on_board yes)
-    (property "Reference" "U5" (id 0) (at 119.38 76.708 0)
+    (property "Reference" "U10" (id 0) (at 119.38 76.708 0)
       (effects (font (size 1.524 1.524)))
     )
@@
   (symbol (lib_id "power:GND") (at 165.608 88.646 90) (unit 1)
     (in_bom yes) (on_board yes) (fields_autoplaced)
-    (property "Reference" "#PWR0231" (id 0) (at 171.958 88.646 0)
+    (property "Reference" "#PWR0122" (id 0) (at 171.958 88.646 0)
       (effects (font (size 1.27 1.27)) hide)
     )
@@
   (symbol (lib_id "Device:C") (at 169.926 75.184 0) (unit 1)
     (in_bom yes) (on_board yes) (fields_autoplaced)
-    (property "Reference" "C15" (id 0) (at 172.847 74.3493 0)
+    (property "Reference" "C87" (id 0) (at 172.847 74.3493 0)
       (effects (font (size 1.27 1.27)) (justify left))
     )

Commit message: All DRC errors cleared after conversion to Kicad V7
Parts:
- removed U10: SN74AHC1G125DBVR, Project_Footprints_Library:SN74AHC1G125DBVR, symbol 1LibBBCTRL:SN74AHC1G125DBVR
- added U28: SN74AHC1G125DBVR, Project_Footprints_Library:SN74AHC1G125DBVR, symbol 1LibBBCTRL:SN74AHC1G125DBVR
Connections:
- net +5V: now also U28.5 (VCC)
- net GND: now also U28.3 (GND)
- net buffer_enable: now also U28.1 (*OE)
- net in: now also U28.2 (A)
- net out: now also U28.4 (Y)
Other:
- moved on the sheet: C87

Commit message: changed level shifter symbol
Parts:
- renumbered U28 to U5
Changed lines of the file:
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@@
   (symbol (lib_name "SN74AHC1G125DBVR_1") (lib_id "1LibBBCTRL:SN74AHC1G125DBVR") (at 109.22 83.82 0) (unit 1)
     (in_bom yes) (on_board yes) (dnp no) (fields_autoplaced)
-    (property "Reference" "U28" (at 125.095 77.47 0)
+    (property "Reference" "U5" (at 125.095 77.47 0)
       (effects (font (size 1.524 1.524)))
     )
@@
       (project "BuildboticsController"
         (path "/7f2164be-b8eb-4dbc-bc7c-152cd10e724f/3adf10c7-5d86-4ad9-b91c-31c97a8ff0e6/e7fccdc6-eaa3-4b15-8a46-061004b9b736"
-          (reference "U28") (unit 1)
+          (reference "U5") (unit 1)
         )
         (path "/7f2164be-b8eb-4dbc-bc7c-152cd10e724f/3adf10c7-5d86-4ad9-b91c-31c97a8ff0e6/7ae97fbc-b32b-4444-aab0-80300a3f3875"
-          (reference "U30") (unit 1)
+          (reference "U17") (unit 1)
         )
         (path "/7f2164be-b8eb-4dbc-bc7c-152cd10e724f/3adf10c7-5d86-4ad9-b91c-31c97a8ff0e6/bcbd1d18-8a29-4a65-81de-0924a31382a8"
-          (reference "U31") (unit 1)
+          (reference "U18") (unit 1)
         )
         (path "/7f2164be-b8eb-4dbc-bc7c-152cd10e724f/3adf10c7-5d86-4ad9-b91c-31c97a8ff0e6/162445ff-f653-4fc4-88d5-5b512f6d58f2"
-          (reference "U32") (unit 1)
+          (reference "U19") (unit 1)
         )
         (path "/7f2164be-b8eb-4dbc-bc7c-152cd10e724f/3adf10c7-5d86-4ad9-b91c-31c97a8ff0e6/fc2c8b20-7ced-44e1-9bd0-0c1868bfc0fe"
-          (reference "U33") (unit 1)
+          (reference "U20") (unit 1)
         )
         (path "/7f2164be-b8eb-4dbc-bc7c-152cd10e724f/3adf10c7-5d86-4ad9-b91c-31c97a8ff0e6/76c04cd0-8257-4c7d-b878-52697c143c99"
-          (reference "U34") (unit 1)
+          (reference "U21") (unit 1)
         )
         (path "/7f2164be-b8eb-4dbc-bc7c-152cd10e724f/3adf10c7-5d86-4ad9-b91c-31c97a8ff0e6/f01e92d1-3ebb-4869-8789-d360c912a5d8"
-          (reference "U35") (unit 1)
+          (reference "U22") (unit 1)
         )
         (path "/7f2164be-b8eb-4dbc-bc7c-152cd10e724f/3adf10c7-5d86-4ad9-b91c-31c97a8ff0e6/22f513e1-2d0b-42a3-93b9-7d1fc0f3e7ae"
-          (reference "U36") (unit 1)
+          (reference "U23") (unit 1)
         )
         (path "/7f2164be-b8eb-4dbc-bc7c-152cd10e724f/3adf10c7-5d86-4ad9-b91c-31c97a8ff0e6/861306e3-ae66-4edf-a865-56b7a91ad832"
-          (reference "U37") (unit 1)
+          (reference "U24") (unit 1)
         )
         (path "/7f2164be-b8eb-4dbc-bc7c-152cd10e724f/3adf10c7-5d86-4ad9-b91c-31c97a8ff0e6/866a1e77-3898-4675-ae7e-206edd135015"
-          (reference "U38") (unit 1)
+          (reference "U13") (unit 1)
         )
         (path "/7f2164be-b8eb-4dbc-bc7c-152cd10e724f/3adf10c7-5d86-4ad9-b91c-31c97a8ff0e6/3cd259a8-cc54-4876-80f3-884a068e413a"
-          (reference "U39") (unit 1)
+          (reference "U14") (unit 1)
         )
         (path "/7f2164be-b8eb-4dbc-bc7c-152cd10e724f/3adf10c7-5d86-4ad9-b91c-31c97a8ff0e6/58bfc332-8446-46b1-b9bf-8a457c28bb3e"
-          (reference "U40") (unit 1)
+          (reference "U15") (unit 1)
         )
         (path "/7f2164be-b8eb-4dbc-bc7c-152cd10e724f/3adf10c7-5d86-4ad9-b91c-31c97a8ff0e6/2271974a-e966-4a72-869e-f0dde9603f54"
-          (reference "U41") (unit 1)
+          (reference "U26") (unit 1)
         )
         (path "/7f2164be-b8eb-4dbc-bc7c-152cd10e724f/15e1e1b6-b278-4e13-8221-f9f8917bc709/0f0648da-b777-4b86-9593-c9dad3aa2b60"
-          (reference "U42") (unit 1)
+          (reference "U10") (unit 1)
         )
         (path "/7f2164be-b8eb-4dbc-bc7c-152cd10e724f/7b65f6db-5358-4955-b729-25fdf7672490/db1c02e9-6be9-4c02-93db-34d7e8ec71c4"
-          (reference "U43") (unit 1)
+          (reference "U27") (unit 1)
         )
       )
