File: level_shifter.kicad_sch (KiCad schematic)
At the start: 2 parts, among them U5 SN74AHC1G125DBVR

Commit message: Replaced D6 with previous part and corrected R13 footprint
Parts:
- renumbered C87 to C92
Changed lines of the file:
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@@
   (symbol (lib_id "power:GND") (at 143.51 87.63 90) (unit 1)
     (in_bom yes) (on_board yes) (dnp no) (fields_autoplaced)
-    (property "Reference" "#PWR0122" (at 149.86 87.63 0)
+    (property "Reference" "#PWR08" (at 149.86 87.63 0)
       (effects (font (size 1.27 1.27)) hide)
     )
@@
   (symbol (lib_name "GND_1") (lib_id "power:GND") (at 147.32 69.85 0) (mirror x) (unit 1)
     (in_bom yes) (on_board yes) (dnp no) (fields_autoplaced)
-    (property "Reference" "#PWR0121" (at 147.32 63.5 0)
+    (property "Reference" "#PWR09" (at 147.32 63.5 0)
       (effects (font (size 1.27 1.27)) hide)
     )
@@
   (symbol (lib_id "Device:C") (at 147.32 74.93 0) (unit 1)
     (in_bom yes) (on_board yes) (dnp no) (fields_autoplaced)
-    (property "Reference" "C87" (at 150.241 74.0953 0)
+    (property "Reference" "C92" (at 150.241 74.0953 0)
       (effects (font (size 1.27 1.27)) (justify left))
     )
